File: Laser Diode Breakout/Laser_Diode_Breakout/Laser_Diode_Breakout.kicad_sch (KiCad schematic)
At the start: 7 parts, among them Q1 BSS138, Q2 BSS138

Commit message: set footprints for most of laser diode breakout
Parts:
- Conn1: footprint (none) -> MRDT_Connectors:MOLEX_SL_04_Vertical
- D2: footprint (none) -> RamanDiodes:PLT5520B - 520nm
- R1: footprint (none) -> Resistor_SMD:R_2512_6332Metric_Pad1.40x3.35mm_HandSolder
- R2: footprint (none) -> Resistor_SMD:R_1206_3216Metric_Pad1.30x1.75mm_HandSolder
Changed lines of the file:
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@@
       (effects (font (size 1.27 1.27)))
     )
-    (property "Footprint" "" (at 86.36 69.85 0)
+    (property "Footprint" "RamanDiodes:PLT5520B - 520nm" (at 86.36 69.85 0)
       (effects (font (size 1.27 1.27)) hide)
     )
@@
       (effects (font (size 1.27 1.27)))
     )
-    (property "Footprint" "" (at 81.28 66.548 90)
+    (property "Footprint" "Resistor_SMD:R_2512_6332Metric_Pad1.40x3.35mm_HandSolder" (at 81.28 66.548 90)
       (effects (font (size 1.27 1.27)) hide)
     )
@@
       (effects (font (size 1.524 1.524)))
     )
-    (property "Footprint" "" (at 40.64 36.83 0)
+    (property "Footprint" "MRDT_Connectors:MOLEX_SL_04_Vertical" (at 40.64 36.83 0)
       (effects (font (size 1.524 1.524)) hide)
     )
@@
       (effects (font (size 1.27 1.27)))
     )
-    (property "Footprint" "" (at 41.91 62.992 90)
-      (effects (font (size 1.27 1.27)) hide)
-    )
+    (property "Footprint" "Resistor_SMD:R_1206_3216Metric_Pad1.30x1.75mm_HandSolder" (at 41.91 62.992 90)
+      (effects (font (size 1.27 1.27)) hide)
+    )
