File: Laser Diode Breakout/Laser_Diode_Breakout/Laser_Diode_Breakout.kicad_pcb (KiCad board)
At the start: 2 copper layers, 29.2 x 35.6 mm, 9 parts, among them Q1 BSS138, Q2 BSS138

Commit message: added ground plane to diode board
Parts:
- turned Q1 to 0 degrees
- turned Q2 to 0 degrees
Routing:
- net GND: track 20.0 -> 0.00 mm, vias 0 -> 4
- net Red_LED: track 17.7 -> 24.6 mm
- net Net-(D1-K): track 9.34 -> 7.48 mm, vias 1 -> 0
- net Green_LED: track 10.3 -> 12.0 mm
- net Net-(D2-K): track 11.6 -> 9.99 mm, vias 1 -> 0
- added copper zone on B.Cu, net GND
- added copper zone on F.Cu, net GND
Changed lines of the file:
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@@
         (effects (font (size 1 1) (thickness 0.15)))
     )
-    (fp_text value "785nm Laser Diode" (at -17.78 3.56) (layer "F.Fab")
+    (fp_text value "785nm Laser Diode" (at 1.27 -2.4) (layer "F.Fab")
         (effects (font (size 1 1) (thickness 0.15)))
     )
@@
   )
   (footprint "Package_TO_SOT_SMD:SOT-23" (layer "B.Cu")
-    (at 35.56 44.45 90)
+    (at 35.56 44.45)
     (descr "SOT, 3 Pin (https://www.jedec.org/system/files/docs/to-236h.pdf variant AB), generated with kicad-footprint-generator ipc_gullwing_generator.py")
     (tags "SOT TO_SOT_SMD")
@@
     (property "ki_keywords" "N-Channel MOSFET")
     (attr smd)
-    (fp_text reference "Q1" (at 0 2.4 90) (layer "B.SilkS")
-        (effects (font (size 1 1) (thickness 0.15)) (justify mirror))
-    )
-    (fp_text value "BSS138" (at 0 -2.4 90) (layer "B.Fab")
-        (effects (font (size 1 1) (thickness 0.15)) (justify mirror))
-    )
-    (fp_text user "${REFERENCE}" (at 0 0 90) (layer "B.Fab")
+    (fp_text reference "Q1" (at 0 2.4) (layer "B.SilkS")
+        (effects (font (size 1 1) (thickness 0.15)) (justify mirror))
+    )
+    (fp_text value "BSS138" (at 0 -2.4) (layer "B.Fab")
+        (effects (font (size 1 1) (thickness 0.15)) (justify mirror))
+    )
+    (fp_text user "${REFERENCE}" (at 0 0) (layer "B.Fab")
         (effects (font (size 0.32 0.32) (thickness 0.05)) (justify mirror))
     )
@@
     (fp_line (start 0.65 1.45) (end 0.65 -1.45)
       (stroke (width 0.1) (type solid)) (layer "B.Fab"))
-    (pad "1" smd roundrect (at -0.9375 0.95 90) (size 1.475 0.6) (layers "B.Cu" "B.Paste" "B.Mask") (roundrect_rratio 0.25)
+    (pad "1" smd roundrect (at -0.9375 0.95) (size 1.475 0.6) (layers "B.Cu" "B.Paste" "B.Mask") (roundrect_rratio 0.25)
       (net 3 "Green_LED") (pinfunction "G") (pintype "input"))
-    (pad "2" smd roundrect (at -0.9375 -0.95 90) (size 1.475 0.6) (layers "B.Cu" "B.Paste" "B.Mask") (roundrect_rratio 0.25)
+    (pad "2" smd roundrect (at -0.9375 -0.95) (size 1.475 0.6) (layers "B.Cu" "B.Paste" "B.Mask") (roundrect_rratio 0.25)
       (net 4 "GND") (pinfunction "S") (pintype "passive"))
-    (pad "3" smd roundrect (at 0.9375 0 90) (size 1.475 0.6) (layers "B.Cu" "B.Paste" "B.Mask") (roundrect_rratio 0.25)
+    (pad "3" smd roundrect (at 0.9375 0) (size 1.475 0.6) (layers "B.Cu" "B.Paste" "B.Mask") (roundrect_rratio 0.25)
       (net 5 "Net-(D2-K)") (pinfunction "D") (pintype "passive"))
     (model "${KICAD6_3DMODEL_DIR}/Package_TO_SOT_SMD.3dshapes/SOT-23.wrl"
@@
   )
   (footprint "Package_TO_SOT_SMD:SOT-23" (layer "B.Cu")
-    (at 35.56 50.8 90)
+    (at 35.56 50.8)
     (descr "SOT, 3 Pin (https://www.jedec.org/system/files/docs/to-236h.pdf variant AB), generated with kicad-footprint-generator ipc_gullwing_generator.py")
     (tags "SOT TO_SOT_SMD")
@@
     (property "ki_keywords" "N-Channel MOSFET")
     (attr smd)
-    (fp_text reference "Q2" (at 0 2.4 90) (layer "B.SilkS")
-        (effects (font (size 1 1) (thickness 0.15)) (justify mirror))
-    )
-    (fp_text value "BSS138" (at 0 -2.4 90) (layer "B.Fab")
-        (effects (font (size 1 1) (thickness 0.15)) (justify mirror))
-    )
-    (fp_text user "${REFERENCE}" (at 0 0 90) (layer "B.Fab")
+    (fp_text reference "Q2" (at 0 2.4) (layer "B.SilkS")
+        (effects (font (size 1 1) (thickness 0.15)) (justify mirror))
+    )
+    (fp_text value "BSS138" (at 0 -2.4) (layer "B.Fab")
+        (effects (font (size 1 1) (thickness 0.15)) (justify mirror))
+    )
+    (fp_text user "${REFERENCE}" (at 0 0) (layer "B.Fab")
         (effects (font (size 0.32 0.32) (thickness 0.05)) (justify mirror))
     )
@@
     (fp_line (start 0.65 1.45) (end 0.65 -1.45)
       (stroke (width 0.1) (type solid)) (layer "B.Fab"))
-    (pad "1" smd roundrect (at -0.9375 0.95 90) (size 1.475 0.6) (layers "B.Cu" "B.Paste" "B.Mask") (roundrect_rratio 0.25)
+    (pad "1" smd roundrect (at -0.9375 0.95) (size 1.475 0.6) (layers "B.Cu" "B.Paste" "B.Mask") (roundrect_rratio 0.25)
       (net 2 "Red_LED") (pinfunction "G") (pintype "input"))
-    (pad "2" smd roundrect (at -0.9375 -0.95 90) (size 1.475 0.6) (layers "B.Cu" "B.Paste" "B.Mask") (roundrect_rratio 0.25)
+    (pad "2" smd roundrect (at -0.9375 -0.95) (size 1.475 0.6) (layers "B.Cu" "B.Paste" "B.Mask") (roundrect_rratio 0.25)
       (net 4 "GND") (pinfunction "S") (pintype "passive"))
-    (pad "3" smd roundrect (at 0.9375 0 90) (size 1.475 0.6) (layers "B.Cu" "B.Paste" "B.Mask") (roundrect_rratio 0.25)
+    (pad "3" smd roundrect (at 0.9375 0) (size 1.475 0.6) (layers "B.Cu" "B.Paste" "B.Mask") (roundrect_rratio 0.25)
       (net 7 "Net-(D1-K)") (pinfunction "D") (pintype "passive"))
     (model "${KICAD6_3DMODEL_DIR}/Package_TO_SOT_SMD.3dshapes/SOT-23.wrl"
@@
   (segment (start 51.435 41.275) (end 46.18 36.02) (width 0.25) (layer "B.Cu") (net 1))
   (segment (start 54.21068 41.275) (end 51.435 41.275) (width 0.25) (layer "B.Cu") (net 1))
-  (segment (start 41.37 38.64) (end 40.005 40.005) (width 0.25) (layer "B.Cu") (net 2))
-  (segment (start 41.37 36.02) (end 41.37 38.64) (width 0.25) (layer "B.Cu") (net 2))
-  (segment (start 40.005 40.005) (end 40.005 48.2425) (width 0.25) (layer "B.Cu") (net 2))
-  (segment (start 40.005 48.2425) (end 36.51 51.7375) (width 0.25) (layer "B.Cu") (net 2))
-  (segment (start 38.83 36.02) (end 38.83 43.0675) (width 0.25) (layer "B.Cu") (net 3))
-  (segment (start 38.83 43.0675) (end 36.51 45.3875) (width 0.25) (layer "B.Cu") (net 3))
-  (segment (start 33.02 50.165) (end 34.5925 51.7375) (width 0.25) (layer "B.Cu") (net 4))
-  (segment (start 36.29 36.02) (end 33.02 39.29) (width 0.25) (layer "B.Cu") (net 4))
-  (segment (start 34.5925 51.7375) (end 34.61 51.7375) (width 0.25) (layer "B.Cu") (net 4))
-  (segment (start 33.02 39.29) (end 33.02 43.815) (width 0.25) (layer "B.Cu") (net 4))
-  (segment (start 34.5925 45.3875) (end 33.02 43.815) (width 0.25) (layer "B.Cu") (net 4))
-  (segment (start 34.61 45.3875) (end 34.5925 45.3875) (width 0.25) (layer "B.Cu") (net 4))
-  (segment (start 33.02 43.815) (end 33.02 50.165) (width 0.25) (layer "B.Cu") (net 4))
-  (segment (start 37.465 43.18) (end 39.656 45.371) (width 0.25) (layer "F.Cu") (net 5))
-  (segment (start 39.656 45.371) (end 44.799 45.371) (width 0.25) (layer "F.Cu") (net 5))
-  (segment (start 44.799 45.371) (end 45.72 44.45) (width 0.25) (layer "F.Cu") (net 5))
-  (via (at 37.465 43.18) (size 0.8) (drill 0.4) (layers "F.Cu" "B.Cu") (net 5))
-  (segment (start 35.8925 43.18) (end 35.56 43.5125) (width 0.25) (layer "B.Cu") (net 5))
-  (segment (start 37.465 43.18) (end 35.8925 43.18) (width 0.25) (layer "B.Cu") (net 5))
+  (segment (start 35.839749 34.933) (end 40.283 34.933) (width 0.25) (layer "B.Cu") (net 2))
+  (segment (start 40.283 34.933) (end 41.37 36.02) (width 0.25) (layer "B.Cu") (net 2))
+  (segment (start 34.6225 51.75) (end 33.11 50.2375) (width 0.25) (layer "B.Cu") (net 2))
+  (segment (start 33.11 37.662749) (end 35.839749 34.933) (width 0.25) (layer "B.Cu") (net 2))
+  (segment (start 33.11 50.2375) (end 33.11 37.662749) (width 0.25) (layer "B.Cu") (net 2))
+  (segment (start 34.6225 45.4) (end 33.56 44.3375) (width 0.25) (layer "B.Cu") (net 3))
+  (segment (start 33.56 44.3375) (end 33.56 41.29) (width 0.25) (layer "B.Cu") (net 3))
+  (segment (start 33.56 41.29) (end 38.83 36.02) (width 0.25) (layer "B.Cu") (net 3))
+  (via (at 34.29 47.498) (size 0.8) (drill 0.4) (layers "F.Cu" "B.Cu") (free) (net 4))
+  (via (at 35.052 37.592) (size 0.8) (drill 0.4) (layers "F.Cu" "B.Cu") (free) (net 4))
+  (via (at 35.306 41.656) (size 0.8) (drill 0.4) (layers "F.Cu" "B.Cu") (free) (net 4))
+  (via (at 34.036 39.116) (size 0.8) (drill 0.4) (layers "F.Cu" "B.Cu") (free) (net 4))
+  (segment (start 36.4975 44.45) (end 37.4185 45.371) (width 0.25) (layer "B.Cu") (net 5))
+  (segment (start 44.799 45.371) (end 45.72 44.45) (width 0.25) (layer "B.Cu") (net 5))
+  (segment (start 37.4185 45.371) (end 44.799 45.371) (width 0.25) (layer "B.Cu") (net 5))
   (segment (start 50.29 43.45432) (end 50.28568 43.45) (width 0.25) (layer "B.Cu") (net 6))
   (segment (start 50.28568 43.45) (end 44.72 43.45) (width 0.25) (layer "B.Cu") (net 6))
-  (segment (start 37.084 49.276) (end 39.37 49.276) (width 0.25) (layer "F.Cu") (net 7))
-  (segment (start 39.37 49.276) (end 42.164 52.07) (width 0.25) (layer "F.Cu") (net 7))
-  (segment (start 42.164 52.07) (end 43.44924 52.07) (width 0.25) (layer "F.Cu") (net 7))
-  (via (at 37.084 49.276) (size 0.8) (drill 0.4) (layers "F.Cu" "B.Cu") (net 7))
-  (segment (start 35.56 49.8625) (end 35.56 49.784) (width 0.25) (layer "B.Cu") (net 7))
-  (segment (start 35.56 49.784) (end 36.068 49.276) (width 0.25) (layer "B.Cu") (net 7))
-  (segment (start 36.068 49.276) (end 37.084 49.276) (width 0.25) (layer "B.Cu") (net 7))
+  (segment (start 37.7675 52.07) (end 43.44924 52.07) (width 0.25) (layer "B.Cu") (net 7))
+  (segment (start 36.4975 50.8) (end 37.7675 52.07) (width 0.25) (layer "B.Cu") (net 7))
   (segment (start 51.79 53.34) (end 44.71924 53.34) (width 0.25) (layer "B.Cu") (net 8))
+  (zone (net 4) (net_name "GND") (layers "F&B.Cu") (hatch edge 0.5)
+    (connect_pads (clearance 0.5))
+    (min_thickness 0.25) (filled_areas_thickness no)
+    (fill (thermal_gap 0.5) (thermal_bridge_width 0.5))
+    (polygon
+      (pts
+        (xy 27.178 28.448)
+        (xy 65.278 28.448)
+        (xy 65.532 68.326)
+        (xy 27.178 68.58)
+        (xy 27.178 28.702)
+      )
+    )
+  )
 )
