File: CCD Breakout/Hardware/CCD_Breakout.kicad_sch (KiCad schematic)
At the start: 6 parts, among them J1 Conn_01x03_Pin, U1 ILX511

Commit message: finish ccd
Parts:
- added V1, V2: Via, MRDT_Drill_Holes:4_40_Hole, symbol MRDT_Drill_Holes:Via
Other:
- note added: "Mounting Holes"
Changed lines of the file:
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@@
+    (stroke (width 0) (type default))
+  )
+  (polyline (pts (xy 118.11 12.7) (xy 118.11 35.56))
     (stroke (width 0) (type default))
   )
@@
     (stroke (width 0) (type default))
   )
+  (polyline (pts (xy 97.79 12.7) (xy 118.11 12.7))
+    (stroke (width 0) (type default))
+  )
   (wire (pts (xy 27.94 44.45) (xy 15.24 44.45))
     (stroke (width 0) (type default))
@@
     (stroke (width 0) (type default))
   )
+  (polyline (pts (xy 97.79 13.97) (xy 97.79 12.7))
+    (stroke (width 0) (type default))
+  )
   (wire (pts (xy 15.24 31.75) (xy 27.94 31.75))
     (stroke (width 0) (type default))
@@
     (stroke (width 0) (type default))
   )
+  (polyline (pts (xy 97.79 35.56) (xy 118.11 35.56))
+    (stroke (width 0) (type default))
+  )
   (polyline (pts (xy 55.88 63.5) (xy 12.7 63.5))
     (stroke (width 0) (type default))
@@
   )
   (wire (pts (xy 15.24 26.67) (xy 15.24 20.32))
+    (stroke (width 0) (type default))
+  )
+  (polyline (pts (xy 97.79 13.97) (xy 97.79 35.56))
     (stroke (width 0) (type default))
   )
@@
   )
   (text "CCD" (at 16.51 60.96 0)
+    (effects (font (size 2.54 2.54)) (justify left bottom))
+  )
+  (text "Mounting\n  Holes" (at 99.06 21.59 0)
     (effects (font (size 2.54 2.54)) (justify left bottom))
   )
@@
         )
       )
+    )
+  )
+  (symbol (lib_id "MRDT_Drill_Holes:Via") (at 106.68 31.75 0) (unit 1)
+    (in_bom yes) (on_board yes) (dnp no) (fields_autoplaced)
+    (property "Reference" "V2" (at 109.22 30.48 0)
+      (effects (font (size 1.524 1.524)) (justify left))
+    )
+    (property "Value" "Via" (at 109.22 33.02 0)
+      (effects (font (size 1.524 1.524)) (justify left))
+    )
+    (property "Footprint" "MRDT_Drill_Holes:4_40_Hole" (at 106.68 31.75 0)
+      (effects (font (size 1.524 1.524)) hide)
+    )
+    (property "Datasheet" "" (at 106.68 31.75 0)
+      (effects (font (size 1.524 1.524)) hide)
+    )
+    (pin "1")
+    (instances
+      (project "CCD_Breakout"
+        (path "/64b006a0-b432-4c05-bc21-eb3325874dfb"
+          (reference "V2") (unit 1)
+        )
+      )
+      (project "Laser_Diode_Breakout"
+        (path "/c855c228-4e5d-4dfd-9922-c2d1c9f93d6f"
+          (reference "V2") (unit 1)
+        )
+      )
+      (project "Raman_Spectrometer_Board"
+        (path "/dd57774e-6364-4f58-a24d-9970470de2f9"
+          (reference "V2") (unit 1)
+        )
+      )
+    )
+  )
+  (symbol (lib_id "MRDT_Drill_Holes:Via") (at 106.68 25.4 0) (unit 1)
+    (in_bom yes) (on_board yes) (dnp no) (fields_autoplaced)
+    (property "Reference" "V1" (at 109.22 24.13 0)
+      (effects (font (size 1.524 1.524)) (justify left))
+    )
+    (property "Value" "Via" (at 109.22 26.67 0)
+      (effects (font (size 1.524 1.524)) (justify left))
+    )
+    (property "Footprint" "MRDT_Drill_Holes:4_40_Hole" (at 106.68 25.4 0)
+      (effects (font (size 1.524 1.524)) hide)
+    )
+    (property "Datasheet" "" (at 106.68 25.4 0)
+      (effects (font (size 1.524 1.524)) hide)
+    )
+    (pin "1")
+    (instances
+      (project "CCD_Breakout"
+        (path "/64b006a0-b432-4c05-bc21-eb3325874dfb"
+          (reference "V1") (unit 1)
+        )
+      )
+      (project "Laser_Diode_Breakout"
+        (path "/c855c228-4e5d-4dfd-9922-c2d1c9f93d6f"
+          (reference "V1") (unit 1)
+        )
+      )
+      (project "Raman_Spectrometer_Board"
+        (path "/dd57774e-6364-4f58-a24d-9970470de2f9"
+          (reference "V1") (unit 1)
+        )
+      )

Commit message: finish ccd board
Parts:
- C3: footprint Capacitor_SMD:C_0201_0603Metric_Pad0.64x0.40mm_HandSolder -> Capacitor_SMD:C_0603_1608Metric_Pad1.08x0.95mm_HandSolder
Changed lines of the file:
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@@
       (effects (font (size 1.27 1.27)) (justify right))
     )
-    (property "Footprint" "Capacitor_SMD:C_0201_0603Metric_Pad0.64x0.40mm_HandSolder" (at 75.2348 24.13 0)
+    (property "Footprint" "Capacitor_SMD:C_0603_1608Metric_Pad1.08x0.95mm_HandSolder" (at 75.2348 24.13 0)
       (effects (font (size 1.27 1.27)) hide)
     )
