File: Laser Diode Breakout/Hardware/Laser_Diode_Breakout.kicad_sch (KiCad schematic)
At the start: 9 parts, among them Q1 BSS138, Q2 BSS138

Commit message: finish diode breakout changes
Parts:
- added V3, V4: Via, MRDT_Drill_Holes:4_40_Hole, symbol MRDT_Drill_Holes:Via
- D1: value 785nm Laser Diode -> 782nm Laser Diode
Other:
- moved on the sheet: V1, V2
Changed lines of the file:
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@@
     )
   )
-  (symbol (lib_id "MRDT_Drill_Holes:Via") (at 96.52 30.48 0) (unit 1)
-    (in_bom yes) (on_board yes) (dnp no) (fields_autoplaced)
-    (property "Reference" "V1" (at 99.06 29.21 0)
-      (effects (font (size 1.524 1.524)) (justify left))
-    )
-    (property "Value" "Via" (at 99.06 31.75 0)
-      (effects (font (size 1.524 1.524)) (justify left))
-    )
-    (property "Footprint" "MRDT_Drill_Holes:4_40_Hole" (at 96.52 30.48 0)
-      (effects (font (size 1.524 1.524)) hide)
-    )
-    (property "Datasheet" "" (at 96.52 30.48 0)
+  (symbol (lib_id "MRDT_Drill_Holes:Via") (at 92.71 30.48 0) (unit 1)
+    (in_bom yes) (on_board yes) (dnp no) (fields_autoplaced)
+    (property "Reference" "V1" (at 95.25 29.21 0)
+      (effects (font (size 1.524 1.524)) (justify left))
+    )
+    (property "Value" "Via" (at 95.25 31.75 0)
+      (effects (font (size 1.524 1.524)) (justify left))
+    )
+    (property "Footprint" "MRDT_Drill_Holes:4_40_Hole" (at 92.71 30.48 0)
+      (effects (font (size 1.524 1.524)) hide)
+    )
+    (property "Datasheet" "" (at 92.71 30.48 0)
       (effects (font (size 1.524 1.524)) hide)
     )
@@
     )
   )
+  (symbol (lib_id "MRDT_Drill_Holes:Via") (at 101.6 30.48 0) (unit 1)
+    (in_bom yes) (on_board yes) (dnp no) (fields_autoplaced)
+    (property "Reference" "V3" (at 104.14 29.21 0)
+      (effects (font (size 1.524 1.524)) (justify left))
+    )
+    (property "Value" "Via" (at 104.14 31.75 0)
+      (effects (font (size 1.524 1.524)) (justify left))
+    )
+    (property "Footprint" "MRDT_Drill_Holes:4_40_Hole" (at 101.6 30.48 0)
+      (effects (font (size 1.524 1.524)) hide)
+    )
+    (property "Datasheet" "" (at 101.6 30.48 0)
+      (effects (font (size 1.524 1.524)) hide)
+    )
+    (pin "1")
+    (instances
+      (project "Laser_Diode_Breakout"
+        (path "/c855c228-4e5d-4dfd-9922-c2d1c9f93d6f"
+          (reference "V3") (unit 1)
+        )
+      )
+      (project "Raman_Spectrometer_Board"
+        (path "/dd57774e-6364-4f58-a24d-9970470de2f9"
+          (reference "V1") (unit 1)
+        )
+      )
+    )
+  )
   (symbol (lib_id "power:GND") (at 86.36 86.36 0) (unit 1)
     (in_bom yes) (on_board yes) (dnp no) (fields_autoplaced)
@@
       (effects (font (size 1.27 1.27)) (justify left))
     )
-    (property "Value" "785nm Laser Diode" (at 49.53 72.7075 90)
+    (property "Value" "782nm Laser Diode" (at 49.53 72.7075 90)
       (effects (font (size 1.27 1.27)) (justify left))
     )
@@
     )
   )
+  (symbol (lib_id "MRDT_Drill_Holes:Via") (at 101.6 36.83 0) (unit 1)
+    (in_bom yes) (on_board yes) (dnp no) (fields_autoplaced)
+    (property "Reference" "V4" (at 104.14 35.56 0)
+      (effects (font (size 1.524 1.524)) (justify left))
+    )
+    (property "Value" "Via" (at 104.14 38.1 0)
+      (effects (font (size 1.524 1.524)) (justify left))
+    )
+    (property "Footprint" "MRDT_Drill_Holes:4_40_Hole" (at 101.6 36.83 0)
+      (effects (font (size 1.524 1.524)) hide)
+    )
+    (property "Datasheet" "" (at 101.6 36.83 0)
+      (effects (font (size 1.524 1.524)) hide)
+    )
+    (pin "1")
+    (instances
+      (project "Laser_Diode_Breakout"
+        (path "/c855c228-4e5d-4dfd-9922-c2d1c9f93d6f"
+          (reference "V4") (unit 1)
+        )
+      )
+      (project "Raman_Spectrometer_Board"
+        (path "/dd57774e-6364-4f58-a24d-9970470de2f9"
+          (reference "V2") (unit 1)
+        )
+      )
+    )
+  )
   (symbol (lib_id "power:+12V") (at 36.83 63.5 0) (unit 1)
     (in_bom yes) (on_board yes) (dnp no) (fields_autoplaced)
@@
     )
   )
-  (symbol (lib_id "MRDT_Drill_Holes:Via") (at 96.52 36.83 0) (unit 1)
-    (in_bom yes) (on_board yes) (dnp no) (fields_autoplaced)
-    (property "Reference" "V2" (at 99.06 35.56 0)
-      (effects (font (size 1.524 1.524)) (justify left))
-    )
-    (property "Value" "Via" (at 99.06 38.1 0)
-      (effects (font (size 1.524 1.524)) (justify left))
-    )
-    (property "Footprint" "MRDT_Drill_Holes:4_40_Hole" (at 96.52 36.83 0)
-      (effects (font (size 1.524 1.524)) hide)
-    )
-    (property "Datasheet" "" (at 96.52 36.83 0)
-      (effects (font (size 1.524 1.524)) hide)
-    )
+  (symbol (lib_id "MRDT_Drill_Holes:Via") (at 92.71 36.83 0) (unit 1)
+    (in_bom yes) (on_board yes) (dnp no) (fields_autoplaced)
+    (property "Reference" "V2" (at 95.25 35.56 0)
+      (effects (font (size 1.524 1.524)) (justify left))
+    )
+    (property "Value" "Via" (at 95.25 38.1 0)
+      (effects (font (size 1.524 1.524)) (justify left))
+    )
+    (property "Footprint" "MRDT_Drill_Holes:4_40_Hole" (at 92.71 36.83 0)
+      (effects (font (size 1.524 1.524)) hide)
+    )
+    (property "Datasheet" "" (at 92.71 36.83 0)
+      (effects (font (size 1.524 1.524)) hide)
+    )

Commit message: add 4.7k resistor to mosfets and regenerate BOM
Parts:
- added R3, R4: 4.7k, Resistor_SMD:R_0603_1608Metric_Pad0.98x0.95mm_HandSolder, symbol Device:R
Connections:
- net GND: now also R3.2, R4.2
- net Green_LED: now also R3.1
- net Red_LED: now also R4.1
Changed lines of the file:
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@@
 (kicad_sch (version 20230121) (generator eeschema)
   (paper "User" 139.7 139.7)
+  (junction (at 38.1 80.01) (diameter 0) (color 0 0 0 0)
+  )
+  (junction (at 77.47 80.01) (diameter 0) (color 0 0 0 0)
+  )
+  (junction (at 46.99 86.36) (diameter 0) (color 0 0 0 0)
+  )
+  (junction (at 86.36 86.36) (diameter 0) (color 0 0 0 0)
+  )
+  (wire (pts (xy 38.1 80.01) (xy 39.37 80.01))
+    (stroke (width 0) (type default))
+  )
   (wire (pts (xy 45.72 27.94) (xy 46.99 27.94))
     (stroke (width 0) (type default))
@@
     (stroke (width 0) (type default))
   )
-  (polyline (pts (xy 33.02 43.18) (xy 73.66 43.18))
+  (polyline (pts (xy 30.48 43.18) (xy 73.66 43.18))
     (stroke (width 0) (type default))
   )
@@
     (stroke (width 0) (type default))
   )
+  (wire (pts (xy 45.72 86.36) (xy 46.99 86.36))
+    (stroke (width 0) (type default))
+  )
+  (wire (pts (xy 85.09 86.36) (xy 86.36 86.36))
+    (stroke (width 0) (type default))
+  )
   (polyline (pts (xy 110.49 41.91) (xy 110.49 17.78))
     (stroke (width 0) (type default))
@@
     (stroke (width 0) (type default))
   )
+  (wire (pts (xy 77.47 80.01) (xy 77.47 86.36))
+    (stroke (width 0) (type default))
+  )
+  (wire (pts (xy 46.99 86.36) (xy 46.99 87.63))
+    (stroke (width 0) (type default))
+  )
   (wire (pts (xy 86.36 64.77) (xy 86.36 66.04))
     (stroke (width 0) (type default))
   )
+  (wire (pts (xy 76.2 80.01) (xy 77.47 80.01))
+    (stroke (width 0) (type default))
+  )
+  (wire (pts (xy 36.83 80.01) (xy 38.1 80.01))
+    (stroke (width 0) (type default))
+  )
+  (wire (pts (xy 46.99 85.09) (xy 46.99 86.36))
+    (stroke (width 0) (type default))
+  )
+  (wire (pts (xy 38.1 80.01) (xy 38.1 86.36))
+    (stroke (width 0) (type default))
+  )
+  (polyline (pts (xy 114.3 46.99) (xy 114.3 93.98))
+    (stroke (width 0) (type default))
+  )
+  (wire (pts (xy 86.36 86.36) (xy 86.36 87.63))
+    (stroke (width 0) (type default))
+  )
+  (polyline (pts (xy 86.36 17.78) (xy 86.36 41.91))
+    (stroke (width 0) (type default))
+  )
+  (wire (pts (xy 36.83 63.5) (xy 36.83 64.77))
+    (stroke (width 0) (type default))
+  )
+  (polyline (pts (xy 86.36 41.91) (xy 110.49 41.91))
+    (stroke (width 0) (type default))
+  )
   (wire (pts (xy 77.47 80.01) (xy 78.74 80.01))
     (stroke (width 0) (type default))
   )
-  (wire (pts (xy 38.1 80.01) (xy 39.37 80.01))
-    (stroke (width 0) (type default))
-  )
-  (wire (pts (xy 46.99 85.09) (xy 46.99 86.36))
-    (stroke (width 0) (type default))
-  )
-  (polyline (pts (xy 114.3 46.99) (xy 114.3 93.98))
-    (stroke (width 0) (type default))
-  )
-  (polyline (pts (xy 86.36 17.78) (xy 86.36 41.91))
-    (stroke (width 0) (type default))
-  )
-  (wire (pts (xy 36.83 63.5) (xy 36.83 64.77))
-    (stroke (width 0) (type default))
-  )
-  (polyline (pts (xy 86.36 41.91) (xy 110.49 41.91))
-    (stroke (width 0) (type default))
-  )
   (polyline (pts (xy 16.51 46.99) (xy 114.3 46.99))
     (stroke (width 0) (type default))
@@
     (stroke (width 0) (type default))
   )
-  (polyline (pts (xy 33.02 17.78) (xy 73.66 17.78))
+  (polyline (pts (xy 30.48 17.78) (xy 73.66 17.78))
     (stroke (width 0) (type default))
   )
@@
     (stroke (width 0) (type default))
   )
-  (polyline (pts (xy 33.02 17.78) (xy 33.02 43.18))
+  (polyline (pts (xy 30.48 17.78) (xy 30.48 43.18))
     (stroke (width 0) (type default))
   )
@@
     )
   )
-  (global_label "Red_LED" (shape input) (at 38.1 80.01 180) (fields_autoplaced)
+  (global_label "Red_LED" (shape input) (at 36.83 80.01 180) (fields_autoplaced)
     (effects (font (size 1.27 1.27)) (justify right))
-    (property "Intersheetrefs" "${INTERSHEET_REFS}" (at 27.1925 80.01 0)
+    (property "Intersheetrefs" "${INTERSHEET_REFS}" (at 25.9225 80.01 0)
       (effects (font (size 1.27 1.27)) (justify right) hide)
     )
   )
-  (global_label "Green_LED" (shape input) (at 77.47 80.01 180) (fields_autoplaced)
+  (global_label "Green_LED" (shape input) (at 76.2 80.01 180) (fields_autoplaced)
     (effects (font (size 1.27 1.27)) (justify right))
-    (property "Intersheetrefs" "${INTERSHEET_REFS}" (at 64.6877 80.01 0)
+    (property "Intersheetrefs" "${INTERSHEET_REFS}" (at 63.4177 80.01 0)
       (effects (font (size 1.27 1.27)) (justify right) hide)
     )
@@
     )
   )
-  (symbol (lib_id "power:GND") (at 46.99 86.36 0) (unit 1)
-    (in_bom yes) (on_board yes) (dnp no) (fields_autoplaced)
-    (property "Reference" "#PWR05" (at 46.99 92.71 0)
-      (effects (font (size 1.27 1.27)) hide)
-    )
-    (property "Value" "GND" (at 46.99 91.44 0)
-      (effects (font (size 1.27 1.27)))
-    )
-    (property "Footprint" "" (at 46.99 86.36 0)
-      (effects (font (size 1.27 1.27)) hide)
-    )
-    (property "Datasheet" "" (at 46.99 86.36 0)
+  (symbol (lib_id "power:GND") (at 46.99 87.63 0) (unit 1)
+    (in_bom yes) (on_board yes) (dnp no) (fields_autoplaced)
+    (property "Reference" "#PWR05" (at 46.99 93.98 0)
+      (effects (font (size 1.27 1.27)) hide)
+    )
+    (property "Value" "GND" (at 46.99 92.71 0)
+      (effects (font (size 1.27 1.27)))
+    )
+    (property "Footprint" "" (at 46.99 87.63 0)
+      (effects (font (size 1.27 1.27)) hide)
+    )
+    (property "Datasheet" "" (at 46.99 87.63 0)
       (effects (font (size 1.27 1.27)) hide)
     )
@@
         (path "/c855c228-4e5d-4dfd-9922-c2d1c9f93d6f"
           (reference "Q2") (unit 1)
+        )
+      )
+    )
+  )
+  (symbol (lib_id "Device:R") (at 81.28 86.36 90) (unit 1)
+    (in_bom yes) (on_board yes) (dnp no)
+    (property "Reference" "R3" (at 81.28 83.82 90)
+      (effects (font (size 1.27 1.27)))
+    )
+    (property "Value" "4.7k" (at 81.28 86.36 90)
+      (effects (font (size 1.27 1.27)))
+    )
+    (property "Footprint" "Resistor_SMD:R_0603_1608Metric_Pad0.98x0.95mm_HandSolder" (at 81.28 88.138 90)
+      (effects (font (size 1.27 1.27)) hide)
+    )
+    (property "Datasheet" "~" (at 81.28 86.36 0)
+      (effects (font (size 1.27 1.27)) hide)
+    )
+    (pin "1")
+    (pin "2")
+    (instances
+      (project "Laser_Diode_Breakout"
+        (path "/c855c228-4e5d-4dfd-9922-c2d1c9f93d6f"
+          (reference "R3") (unit 1)
+        )
+      )
+      (project "Raman_Spectrometer_Board"
+        (path "/dd57774e-6364-4f58-a24d-9970470de2f9"
+          (reference "R1") (unit 1)
         )
       )
@@
     )
   )
-  (symbol (lib_id "power:GND") (at 86.36 86.36 0) (unit 1)
-    (in_bom yes) (on_board yes) (dnp no) (fields_autoplaced)
-    (property "Reference" "#PWR06" (at 86.36 92.71 0)
-      (effects (font (size 1.27 1.27)) hide)
-    )
-    (property "Value" "GND" (at 86.36 91.44 0)
-      (effects (font (size 1.27 1.27)))
-    )
-    (property "Footprint" "" (at 86.36 86.36 0)
-      (effects (font (size 1.27 1.27)) hide)
-    )
-    (property "Datasheet" "" (at 86.36 86.36 0)
+  (symbol (lib_id "power:GND") (at 86.36 87.63 0) (unit 1)
+    (in_bom yes) (on_board yes) (dnp no) (fields_autoplaced)
+    (property "Reference" "#PWR06" (at 86.36 93.98 0)
+      (effects (font (size 1.27 1.27)) hide)
+    )
+    (property "Value" "GND" (at 86.36 92.71 0)
+      (effects (font (size 1.27 1.27)))
+    )
+    (property "Footprint" "" (at 86.36 87.63 0)
+      (effects (font (size 1.27 1.27)) hide)
+    )
+    (property "Datasheet" "" (at 86.36 87.63 0)
       (effects (font (size 1.27 1.27)) hide)
     )
@@
         )
       )
+    )
+  )
+  (symbol (lib_id "Device:R") (at 41.91 86.36 90) (unit 1)
+    (in_bom yes) (on_board yes) (dnp no)
+    (property "Reference" "R4" (at 41.91 83.82 90)
+      (effects (font (size 1.27 1.27)))
+    )
+    (property "Value" "4.7k" (at 41.91 86.36 90)
+      (effects (font (size 1.27 1.27)))
+    )
+    (property "Footprint" "Resistor_SMD:R_0603_1608Metric_Pad0.98x0.95mm_HandSolder" (at 41.91 88.138 90)
+      (effects (font (size 1.27 1.27)) hide)
+    )
+    (property "Datasheet" "~" (at 41.91 86.36 0)
+      (effects (font (size 1.27 1.27)) hide)
+    )
+    (pin "1")
+    (pin "2")
+    (instances
+      (project "Laser_Diode_Breakout"
+        (path "/c855c228-4e5d-4dfd-9922-c2d1c9f93d6f"
+          (reference "R4") (unit 1)
+        )
+      )
+      (project "Raman_Spectrometer_Board"
+        (path "/dd57774e-6364-4f58-a24d-9970470de2f9"
+          (reference "R1") (unit 1)
+        )
+      )
