File: CCD_Breakout/CCD_Breakout.kicad_pcb (KiCad board)
At the start: 2 copper layers, 11 parts, among them Q1 PNP, U1 ILX511

Commit message: Updated CCD
Parts:
- removed H3, H4: ~, MRDT_Drill_Holes:4_40_Hole
- moved Conn1 2.00 mm to (166.0, 97.7)
- moved C2 1.50 mm to (166.0, 93.0)
- moved R1 1.50 mm to (161.0, 93.0)
- moved C3 1.00 mm to (161.0, 90.0)
- moved H1 1.00 mm to (161.0, 38.5)
- moved H2 1.00 mm to (161.0, 107.0)
- moved Q1 0.94 mm to (155.5, 91.5)
- moved C1 0.50 mm to (166.0, 90.0)
Routing:
- net +5V: track 32.8 -> 28.4 mm
- net CLK: track 35.6 -> 37.6 mm
- net ROG: track 19.3 -> 21.3 mm
- net Vout: track 9.02 -> 10.6 mm
- net Net-(U1-VGG): track 27.5 -> 28.5 mm
- net Net-(Q1-B): track 39.2 -> 40.1 mm
- added copper zone on B.Cu, net GND
- added copper zone on F.Cu, net GND
Other:
- board outline added: 16 x 76.5 mm

Commit message: CCD Changes
Parts:
- moved Conn1 51.5 mm to (114.5, 98.7), turned to 0 degrees
- moved H2 41.5 mm to (119.5, 105.7)
- moved C1 41.5 mm to (124.5, 89.2)
- moved C2 41.5 mm to (124.5, 92.2)
- moved C3 41.5 mm to (119.5, 89.2)
- moved Q1 41.5 mm to (114.0, 90.7)
- moved R1 41.5 mm to (119.5, 92.2)
- moved U1 41.5 mm to (124.5, 44.2)
- moved H1 41.5 mm to (119.5, 38.2)
Routing:
- net +5V: track 28.4 -> 112.8 mm, vias 0 -> 2
- net GND: track 0.00 -> 13.8 mm, vias 0 -> 2
- net Vout: track 10.6 -> 16.5 mm
- net ROG: track 21.3 -> 27.2 mm
- net CLK: track 37.6 -> 43.3 mm

Commit message: cat
Parts:
- moved Conn1 74.8 mm to (66.2, 41.5)
- moved C2 73.9 mm to (66.4, 46.5), turned to 180 degrees
- moved C1 70.4 mm to (66.4, 49.5), turned to 180 degrees
- moved R1 66.4 mm to (71.4, 46.5), turned to 0 degrees
- moved C3 62.4 mm to (71.4, 49.5), turned to 180 degrees
- moved Q1 57.0 mm to (76.3, 48.0), turned to 90 degrees
- moved U1 49.0 mm to (76.2, 52.9)
- moved H1 48.6 mm to (71.2, 32.7)
- moved H2 48.6 mm to (71.2, 100.2)
Routing:
- net ROG: track 27.2 -> 55.7 mm
- net +5V: track 112.8 -> 90.6 mm
- net Net-(Q1-B): track 40.1 -> 23.6 mm
- net GND: track 13.8 -> 0.00 mm, vias 2 -> 1
- net Vout: track 16.5 -> 9.77 mm
- net CLK: track 43.3 -> 37.1 mm
- net Net-(U1-VGG): track 28.5 -> 29.5 mm
Other:
- outline, holes or cut-outs redrawn
