File: Raman Spectrometer Board/Raman_Spectrometer_Board/Raman_Spectrometer_Board.kicad_pcb (KiCad board)
At the start: 2 copper layers, 65.5 x 91.4 mm, 35 parts, among them J1 RJ45_LED_Shielded, Q1 BSS138, Q2 BSS138, Q3 BSS138, Q4 BSS138, SW1 SW_Push, SW2 SW_Push, U1 Teensy4.1_DEV-16771, U2 OKI 12V-5V

Commit message: updated Raman PCB
Parts:
- added Conn11: GimbalA, MRDT_Connectors:MOLEX_SL_03_Vertical, F.Cu at (100.6, 32.0)
- added Conn12: GimbalB, MRDT_Connectors:MOLEX_SL_03_Vertical, F.Cu at (100.6, 43.7)
- Conn10: value Molex_SL_02 -> LimitSwitch3
- Conn7: value Molex_SL_04 -> MotorEncoder
- Conn8: value Molex_SL_02 -> LimitSwitch1
- Conn9: value Molex_SL_02 -> LimitSwitch2
- moved D3 0.91 mm to (90.4, 97.0)
- moved R2 0.91 mm to (86.3, 91.9)
- moved R4 0.91 mm to (86.3, 97.0)
- moved D1 0.91 mm to (90.6, 86.9)
- moved D2 0.91 mm to (90.3, 91.9)
- moved R1 0.91 mm to (86.4, 86.9)
- moved Q1 0.68 mm to (88.1, 31.4)
- moved R3 0.68 mm to (84.7, 33.5)
Connections:
- U1 pad 36: unconnected-(U1-CS2-Pad36) -> GimbalPWM_A
- U1 pad 37: unconnected-(U1-CS3-Pad37) -> GimbalPWM_B
Routing:
- net T-: track 0.00 -> 66.7 mm
- net R+: track 0.00 -> 59.5 mm
- net T+: track 0.00 -> 57.4 mm
- net R-: track 0.00 -> 55.8 mm
- net GimbalPWM_A: track 0.00 -> 30.8 mm, vias 0 -> 1
- net +5V: track 135.1 -> 162.2 mm
- net GimbalPWM_B: track 0.00 -> 20.3 mm, vias 0 -> 1
- net Green_Laser_3.3V: track 42.7 -> 48.0 mm
- net GPIO: track 50.6 -> 53.5 mm
- net +12V: track 78.4 -> 77.6 mm
- net Net-(Q1-D): track 8.79 -> 9.48 mm
Other:
- board text added: "CCD"
- board text added: "Fan"
- board text added: "Gantry"
- board text added: "Gimbal A"
- board text added: "Gimbal B"
- board text added: "Laser"
- board text added: "LimSwitch1"
- board text added: "LimSwitch2"
- board text added: "LimSwitch3"
- board text added: "Motor Encoder"
- board text added: "TOF Sensor"

Commit message: Finished Rev2
Parts:
- moved D1 24.7 mm to (86.9, 111.3), turned to -90 degrees
- moved R1 20.8 mm to (86.9, 107.7), turned to 90 degrees
- moved D2 19.3 mm to (90.2, 111.3), turned to -90 degrees
- moved R2 16.2 mm to (90.2, 107.7), turned to 90 degrees
- moved D3 14.5 mm to (93.2, 111.3), turned to -90 degrees
- moved R4 12.7 mm to (93.2, 107.7), turned to 90 degrees
- moved H4 8.27 mm to (142.7, 112.0), turned to 90 degrees
- moved H3 6.10 mm to (142.7, 23.1)
- moved R3 5.61 mm to (90.2, 34.5), turned to 0 degrees
- moved Conn2 5.59 mm to (142.2, 66.0)
- moved Conn6 5.59 mm to (142.2, 87.9)
- moved Conn10 5.59 mm to (142.5, 54.6)
- moved Conn8 5.59 mm to (142.5, 34.9)
- moved Conn9 5.59 mm to (142.5, 44.7)
- moved H2 5.59 mm to (79.2, 112.0)
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Connections:
- Conn5 pad 2: CCD_Vout -> CCD_CLK_5V
- Conn5 pad 4: CCD_CLK_5V -> CCD_Vout
Routing:
- net +12V: track 77.6 -> 100.3 mm
- net +5V: track 162.2 -> 182.4 mm, vias 2 -> 4
- net Net-(C3-Pad1): track 4.86 -> 18.0 mm, vias 0 -> 1
- net +3.3V: track 223.2 -> 229.9 mm
- net CCD_CLK_5V: track 14.5 -> 20.7 mm, vias 0 -> 1
- net Limit Switch 1: track 24.5 -> 30.4 mm
- net Limit Switch 2: track 17.4 -> 23.1 mm
- net SDA: track 31.6 -> 37.2 mm
- net SCL: track 40.6 -> 46.2 mm
- net PWM: track 8.85 -> 14.4 mm
- net IN_A: track 8.85 -> 14.4 mm
- net CS: track 25.3 -> 30.9 mm
- net SEL: track 8.85 -> 14.4 mm
- net IN_B: track 8.85 -> 14.4 mm
- net Limit Switch 3: track 9.84 -> 15.4 mm
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- added copper zone on B.Cu, net GND
- added copper zone on F.Cu, net GND
Other:
- board size 65.5 x 91.4 mm -> 71.6 x 97 mm
- board text added: "-"
- board text added: "12V"
- board text added: "3V3"
- board text added: "5V"
- board text added: "A"
- board text added: "B"
- board text added: "CLK"
- board text added: "CS"
- board text added: "GND"
- board text added: "IO"
- board text added: "OUT"
- board text added: "PWM"
- board text added: "ROG"
- board text added: "SCL"
- board text added: "SDA"
- board text added: "SEL"

Commit message: Finished Rev2
Parts:
- added J2: Conn_01x03_Pin, Connector_PinHeader_2.54mm:PinHeader_1x03_P2.54mm_Vertical, F.Cu at (108.6, 69.6)
- added J3: Conn_01x03_Pin, Connector_PinHeader_2.54mm:PinHeader_1x03_P2.54mm_Vertical, F.Cu at (103.5, 61.0)
- moved D1 54.8 mm to (141.4, 105.0), turned to 0 degrees
- moved D2 51.8 mm to (141.3, 103.1), turned to 0 degrees
- moved R1 51.0 mm to (137.8, 105.0), turned to 180 degrees
- moved D3 49.1 mm to (141.3, 101.3), turned to 0 degrees
- moved R2 47.8 mm to (137.8, 103.1), turned to 180 degrees
- moved R4 45.0 mm to (137.8, 101.3), turned to 180 degrees
- moved C2 23.2 mm to (90.9, 109.0), turned to 180 degrees
- moved R6 21.6 mm to (106.8, 43.9)
- moved R5 20.9 mm to (106.8, 37.7)
- moved R3 16.9 mm to (106.8, 31.6), turned to 90 degrees
- moved Q1 15.1 mm to (103.3, 31.6)
- moved Q4 14.3 mm to (103.3, 43.9)
- moved Q3 13.2 mm to (103.3, 37.8)
- moved Conn12 12.2 mm to (88.5, 42.2)
- moved Conn11 12.1 mm to (88.5, 31.4)
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Connections:
- U1 pad 38: unconnected-(U1-A14-Pad38) -> STRAIN_GAUGE_2
- U1 pad 39: unconnected-(U1-A15-Pad39) -> STRAIN_GAUGE_1
Routing:
- net +5V: track 182.4 -> 267.5 mm, vias 4 -> 3
- net +12V: track 100.3 -> 146.9 mm, vias 0 -> 2
- net GPIO: track 58.7 -> 31.6 mm, vias 0 -> 1
- net CCD_ROG_5V: track 14.9 -> 41.0 mm, vias 0 -> 1
- net GimbalPWM_B: track 20.3 -> 41.2 mm, vias 1 -> 3
- net FAN_OUT: track 67.6 -> 87.9 mm, vias 1 -> 3
- net GimbalPWM_A: track 30.8 -> 51.0 mm, vias 1 -> 2
- net STRAIN_GAUGE_2: track 0.00 -> 20.1 mm
- net +3.3V: track 229.9 -> 210.9 mm, vias 0 -> 4
- net Net-(Q1-D): track 9.48 -> 25.5 mm
- net Green_Laser_3.3V: track 45.5 -> 30.2 mm
- net STRAIN_GAUGE_1: track 0.00 -> 14.9 mm
- net CCD_CLK_5V: track 20.7 -> 35.0 mm
- net LED: track 82.4 -> 76.3 mm
- net CCD_ROG_3.3V: track 60.1 -> 66.1 mm, vias 1 -> 3
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