File: board/ethernet.kicad_sch (KiCad schematic)
At the start: 0 parts

Commit message: Added Ethernet
Parts:
- added C3: .1uF, symbol Device:C
- added J1: RJ45_LED_Shielded, symbol Connector:RJ45_LED_Shielded
Connections:
- new net: C3.1, J1.2, J1.5
- new net GND: C3.2, J1.8, J1.9, J1.SH
- new net LED: J1.10
- new net R+: J1.4
- new net R-: J1.6
- new net T+: J1.1
- new net T-: J1.3
- no-connect marks 0 -> 3
