File: Raman Spectrometer Board/ethernet.kicad_sch (KiCad schematic)
At the start: 2 parts, among them J1 RJ45_LED_Shielded

Commit message: tof voltages connected
Parts:
- C3: footprint Capacitor_SMD:C_0603_1608Metric_Pad1.08x0.95mm_HandSolder -> (none)
- J1: footprint MRDT_Connectors:RJ45_Teensy -> (none)
Changed lines of the file:
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@@
 			)
 		)
-		(property "Footprint" "MRDT_Connectors:RJ45_Teensy"
+		(property "Footprint" ""
 			(at 157.48 94.615 90)
 			(effects
@@
 			)
 		)
-		(property "Footprint" "Capacitor_SMD:C_0603_1608Metric_Pad1.08x0.95mm_HandSolder"
+		(property "Footprint" ""
 			(at 184.15 95.5548 0)
 			(effects

Commit message: Added footprints to main board
Parts:
- C3: footprint (none) -> Capacitor_SMD:C_0603_1608Metric_Pad1.08x0.95mm_HandSolder
- J1: footprint (none) -> MRDT_Connectors:RJ45_Teensy
Changed lines of the file:
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@@
 			)
 		)
-		(property "Footprint" ""
+		(property "Footprint" "MRDT_Connectors:RJ45_Teensy"
 			(at 157.48 94.615 90)
 			(effects
@@
 			)
 		)
-		(property "Footprint" ""
+		(property "Footprint" "Capacitor_SMD:C_0603_1608Metric_Pad1.08x0.95mm_HandSolder"
 			(at 184.15 95.5548 0)
 			(effects
