File: Raman Spectrometer Board/fanConnector.kicad_sch (KiCad schematic)
At the start: 2 parts, among them Q3 BSS138

Commit message: Added footprints to main board
Parts:
- Conn4: footprint (none) -> MRDT_Connectors:MOLEX_SL_02_Vertical
Changed lines of the file:
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@@
 		(dnp no)
 		(fields_autoplaced yes)
-		(property "Reference" "#PWR027"
+		(property "Reference" "#PWR0102"
 			(at 161.29 92.71 0)
 			(effects
@@
 			(project ""
 				(path "/ab487c59-f066-48f5-a383-99e8eaf806bf/bf499055-0d6c-41cb-ad4c-c2bb3d96cc3f"
-					(reference "#PWR027")
+					(reference "#PWR0102")
 					(unit 1)
 				)
@@
 			)
 		)
-		(property "Footprint" ""
+		(property "Footprint" "MRDT_Connectors:MOLEX_SL_02_Vertical"
 			(at 151.13 87.63 0)
 			(effects
@@
 		(dnp no)
 		(fields_autoplaced yes)
-		(property "Reference" "#PWR026"
+		(property "Reference" "#PWR0101"
 			(at 161.29 119.38 0)
 			(effects
@@
 			(project ""
 				(path "/ab487c59-f066-48f5-a383-99e8eaf806bf/bf499055-0d6c-41cb-ad4c-c2bb3d96cc3f"
-					(reference "#PWR026")
-					(unit 1)
-				)
+					(reference "#PWR0101")
+					(unit 1)
+				)

Commit message: tof voltages connected
Parts:
- Conn4: footprint MRDT_Connectors:MOLEX_SL_02_Vertical -> (none)
Changed lines of the file:
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@@
 		(dnp no)
 		(fields_autoplaced yes)
-		(property "Reference" "#PWR0102"
+		(property "Reference" "#PWR027"
 			(at 161.29 92.71 0)
 			(effects
@@
 			(project ""
 				(path "/ab487c59-f066-48f5-a383-99e8eaf806bf/bf499055-0d6c-41cb-ad4c-c2bb3d96cc3f"
-					(reference "#PWR0102")
+					(reference "#PWR027")
 					(unit 1)
 				)
@@
 			)
 		)
-		(property "Footprint" "MRDT_Connectors:MOLEX_SL_02_Vertical"
+		(property "Footprint" ""
 			(at 151.13 87.63 0)
 			(effects
@@
 		(dnp no)
 		(fields_autoplaced yes)
-		(property "Reference" "#PWR0101"
+		(property "Reference" "#PWR026"
 			(at 161.29 119.38 0)
 			(effects
@@
 			(project ""
 				(path "/ab487c59-f066-48f5-a383-99e8eaf806bf/bf499055-0d6c-41cb-ad4c-c2bb3d96cc3f"
-					(reference "#PWR0101")
-					(unit 1)
-				)
+					(reference "#PWR026")
+					(unit 1)
+				)
