File: Raman Spectrometer Board/oki.kicad_sch (KiCad schematic)
At the start: 3 parts, among them U1 OKI

Commit message: Added footprints to main board
Parts:
- C1, C2: footprint (none) -> Capacitor_SMD:C_0603_1608Metric_Pad1.08x0.95mm_HandSolder
- U1: footprint (none) -> MRDT_Devices:OKI_Horizontal
Changed lines of the file:
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@@
 			)
 		)
-		(property "Footprint" ""
+		(property "Footprint" "MRDT_Devices:OKI_Horizontal"
 			(at 143.51 102.87 0)
 			(effects
@@
 			)
 		)
-		(property "Footprint" ""
+		(property "Footprint" "Capacitor_SMD:C_0603_1608Metric_Pad1.08x0.95mm_HandSolder"
 			(at 138.1252 111.76 0)
 			(effects
@@
 			)
 		)
-		(property "Footprint" ""
+		(property "Footprint" "Capacitor_SMD:C_0603_1608Metric_Pad1.08x0.95mm_HandSolder"
 			(at 171.1452 111.76 0)
 			(effects

Commit message: tof voltages connected
Parts:
- C1, C2: footprint Capacitor_SMD:C_0603_1608Metric_Pad1.08x0.95mm_HandSolder -> (none)
- U1: footprint MRDT_Devices:OKI_Horizontal -> (none)
Changed lines of the file:
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@@
 			)
 		)
-		(property "Footprint" "MRDT_Devices:OKI_Horizontal"
+		(property "Footprint" ""
 			(at 143.51 102.87 0)
 			(effects
@@
 			)
 		)
-		(property "Footprint" "Capacitor_SMD:C_0603_1608Metric_Pad1.08x0.95mm_HandSolder"
+		(property "Footprint" ""
 			(at 138.1252 111.76 0)
 			(effects
@@
 			)
 		)
-		(property "Footprint" "Capacitor_SMD:C_0603_1608Metric_Pad1.08x0.95mm_HandSolder"
+		(property "Footprint" ""
 			(at 171.1452 111.76 0)
 			(effects
