File: Raman Spectrometer Board/servos.kicad_sch (KiCad schematic)
At the start: 0 parts

Commit message: Servo Connectors
This definitely, need to be checked.
Parts:
- added ServoCon2, ServoConn1: Molex_SL_03, symbol MRDT_Connectors:Molex_SL_03
Connections:
- new net +5V: ServoCon2.1, ServoConn1.1
- new net GND: ServoCon2.3, ServoConn1.3
- new net Servo1: ServoConn1.2
- new net Servo2: ServoCon2.2

Commit message: Added footprints to main board
Parts:
- ServoCon2, ServoConn1: footprint (none) -> MRDT_Connectors:MOLEX_SL_03_Vertical
Changed lines of the file:
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@@
 			)
 		)
-		(property "Footprint" ""
+		(property "Footprint" "MRDT_Connectors:MOLEX_SL_03_Vertical"
 			(at 153.67 80.01 0)
 			(effects
@@
 			)
 		)
-		(property "Footprint" ""
+		(property "Footprint" "MRDT_Connectors:MOLEX_SL_03_Vertical"
 			(at 153.67 104.14 0)
 			(effects

Commit message: tof voltages connected
Parts:
- ServoCon2, ServoConn1: footprint MRDT_Connectors:MOLEX_SL_03_Vertical -> (none)
Changed lines of the file:
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@@
 			)
 		)
-		(property "Footprint" "MRDT_Connectors:MOLEX_SL_03_Vertical"
+		(property "Footprint" ""
 			(at 153.67 80.01 0)
 			(effects
@@
 			)
 		)
-		(property "Footprint" "MRDT_Connectors:MOLEX_SL_03_Vertical"
+		(property "Footprint" ""
 			(at 153.67 104.14 0)
 			(effects
