File: Raman Spectrometer Board/canTransciever.kicad_sch (KiCad schematic)
At the start: 17 parts, among them SW2 SW_Push, SW3 SW_Push, U5 ATA6561, U6 ATA6561

Commit message: Began re-laying out laser driver section
Parts:
- renumbered C12 to C14, C13 to C15, C14 to C16, C15 to C17, C16 to C18, C17 to C19, SW2 to SW1, SW3 to SW2, U5 to U6, U6 to U7
Changed lines of the file:
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@@
 		(dnp no)
 		(fields_autoplaced yes)
-		(property "Reference" "#PWR051"
+		(property "Reference" "#PWR056"
 			(at 86.36 35.56 0)
 			(effects
@@
 			(project "RamanSpectrometerBoard"
 				(path "/ab487c59-f066-48f5-a383-99e8eaf806bf/2495d964-2266-4066-961c-06fbcb7a3cda"
-					(reference "#PWR051")
+					(reference "#PWR056")
 					(unit 1)
 				)
@@
 		(dnp no)
 		(fields_autoplaced yes)
-		(property "Reference" "#PWR057"
+		(property "Reference" "#PWR062"
 			(at 190.5 87.63 0)
 			(effects
@@
 			(project "RamanSpectrometerBoard"
 				(path "/ab487c59-f066-48f5-a383-99e8eaf806bf/2495d964-2266-4066-961c-06fbcb7a3cda"
-					(reference "#PWR057")
+					(reference "#PWR062")
 					(unit 1)
 				)
@@
 		(on_board yes)
 		(dnp no)
-		(property "Reference" "C14"
+		(property "Reference" "C16"
 			(at 98.552 58.674 0)
 			(effects
@@
 			(project "RamanSpectrometerBoard"
 				(path "/ab487c59-f066-48f5-a383-99e8eaf806bf/2495d964-2266-4066-961c-06fbcb7a3cda"
-					(reference "C14")
+					(reference "C16")
 					(unit 1)
 				)
@@
 		(on_board yes)
 		(dnp no)
-		(property "Reference" "C12"
+		(property "Reference" "C14"
 			(at 67.818 41.91 0)
 			(effects
@@
 			(project "RamanSpectrometerBoard"
 				(path "/ab487c59-f066-48f5-a383-99e8eaf806bf/2495d964-2266-4066-961c-06fbcb7a3cda"
-					(reference "C12")
+					(reference "C14")
 					(unit 1)
 				)
@@
 		(dnp no)
 		(fields_autoplaced yes)
-		(property "Reference" "#PWR049"
+		(property "Reference" "#PWR054"
 			(at 81.28 35.56 0)
 			(effects
@@
 			(project "RamanSpectrometerBoard"
 				(path "/ab487c59-f066-48f5-a383-99e8eaf806bf/2495d964-2266-4066-961c-06fbcb7a3cda"
-					(reference "#PWR049")
+					(reference "#PWR054")
 					(unit 1)
 				)
@@
 		(on_board yes)
 		(dnp no)
-		(property "Reference" "#PWR060"
+		(property "Reference" "#PWR065"
 			(at 208.28 73.66 0)
 			(effects
@@
 			(project "RamanSpectrometerBoard"
 				(path "/ab487c59-f066-48f5-a383-99e8eaf806bf/2495d964-2266-4066-961c-06fbcb7a3cda"
-					(reference "#PWR060")
+					(reference "#PWR065")
 					(unit 1)
 				)
@@
 		(dnp no)
 		(fields_autoplaced yes)
-		(property "Reference" "#PWR050"
+		(property "Reference" "#PWR055"
 			(at 83.82 87.63 0)
 			(effects
@@
 			(project "RamanSpectrometerBoard"
 				(path "/ab487c59-f066-48f5-a383-99e8eaf806bf/2495d964-2266-4066-961c-06fbcb7a3cda"
-					(reference "#PWR050")
+					(reference "#PWR055")
 					(unit 1)
 				)
@@
 		(on_board yes)
 		(dnp no)
-		(property "Reference" "#PWR048"
+		(property "Reference" "#PWR053"
 			(at 76.2 54.61 0)
 			(effects
@@
 			(project "RamanSpectrometerBoard"
 				(path "/ab487c59-f066-48f5-a383-99e8eaf806bf/2495d964-2266-4066-961c-06fbcb7a3cda"
-					(reference "#PWR048")
+					(reference "#PWR053")
 					(unit 1)
 				)
@@
 		(on_board yes)
 		(dnp no)
-		(property "Reference" "#PWR055"
+		(property "Reference" "#PWR060"
 			(at 182.88 54.61 0)
 			(effects
@@
 			(project "RamanSpectrometerBoard"
 				(path "/ab487c59-f066-48f5-a383-99e8eaf806bf/2495d964-2266-4066-961c-06fbcb7a3cda"
-					(reference "#PWR055")
+					(reference "#PWR060")
 					(unit 1)
 				)
@@
 		(on_board yes)
 		(dnp no)
-		(property "Reference" "#PWR059"
+		(property "Reference" "#PWR064"
 			(at 198.12 54.61 0)
 			(effects
@@
 			(project "RamanSpectrometerBoard"
 				(path "/ab487c59-f066-48f5-a383-99e8eaf806bf/2495d964-2266-4066-961c-06fbcb7a3cda"
-					(reference "#PWR059")
+					(reference "#PWR064")
 					(unit 1)
 				)
@@
 		(dnp no)
 		(fields_autoplaced yes)
-		(property "Reference" "SW2"
+		(property "Reference" "SW1"
 			(at 53.34 167.64 0)
 			(effects
@@
 			(project "RamanSpectrometerBoard"
 				(path "/ab487c59-f066-48f5-a383-99e8eaf806bf/2495d964-2266-4066-961c-06fbcb7a3cda"
-					(reference "SW2")
+					(reference "SW1")
 					(unit 1)
 				)
@@
 		(dnp no)
 		(fields_autoplaced yes)
-		(property "Reference" "C13"
+		(property "Reference" "C15"
 			(at 95.25 41.9099 0)
 			(effects
@@
 			(project "RamanSpectrometerBoard"
 				(path "/ab487c59-f066-48f5-a383-99e8eaf806bf/2495d964-2266-4066-961c-06fbcb7a3cda"
-					(reference "C13")
+					(reference "C15")
 					(unit 1)
 				)
@@
 		(on_board yes)
 		(dnp no)
-		(property "Reference" "#PWR052"
+		(property "Reference" "#PWR057"
 			(at 91.44 54.61 0)
 			(effects
@@
 			(project "RamanSpectrometerBoard"
 				(path "/ab487c59-f066-48f5-a383-99e8eaf806bf/2495d964-2266-4066-961c-06fbcb7a3cda"
-					(reference "#PWR052")
+					(reference "#PWR057")
 					(unit 1)
 				)
@@
 		(dnp no)
 		(fields_autoplaced yes)
-		(property "Reference" "U6"
+		(property "Reference" "U7"
 			(at 192.6433 74.93 0)
 			(effects
@@
 			(project ""
 				(path "/ab487c59-f066-48f5-a383-99e8eaf806bf/2495d964-2266-4066-961c-06fbcb7a3cda"
-					(reference "U6")
+					(reference "U7")
 					(unit 1)
 				)
@@
 		(on_board yes)
 		(dnp no)
-		(property "Reference" "#PWR053"
+		(property "Reference" "#PWR058"
 			(at 101.6 73.66 0)
 			(effects
@@
 			(project "RamanSpectrometerBoard"
 				(path "/ab487c59-f066-48f5-a383-99e8eaf806bf/2495d964-2266-4066-961c-06fbcb7a3cda"
-					(reference "#PWR053")
+					(reference "#PWR058")
 					(unit 1)
 				)
@@
 		(dnp no)
 		(fields_autoplaced yes)
-		(property "Reference" "C16"
+		(property "Reference" "C18"
 			(at 201.93 41.9099 0)
 			(effects
@@
 			(project "RamanSpectrometerBoard"
 				(path "/ab487c59-f066-48f5-a383-99e8eaf806bf/2495d964-2266-4066-961c-06fbcb7a3cda"
-					(reference "C16")
+					(reference "C18")
 					(unit 1)
 				)
@@
 		(on_board yes)
 		(dnp no)
-		(property "Reference" "C15"
+		(property "Reference" "C17"
 			(at 174.498 41.91 0)
 			(effects
@@
 			(project "RamanSpectrometerBoard"
 				(path "/ab487c59-f066-48f5-a383-99e8eaf806bf/2495d964-2266-4066-961c-06fbcb7a3cda"
-					(reference "C15")
+					(reference "C17")
 					(unit 1)
 				)
@@
 		(dnp no)
 		(fields_autoplaced yes)
-		(property "Reference" "U5"
+		(property "Reference" "U6"
 			(at 85.9633 74.93 0)
 			(effects
@@
 			(project "RamanSpectrometerBoard"
 				(path "/ab487c59-f066-48f5-a383-99e8eaf806bf/2495d964-2266-4066-961c-06fbcb7a3cda"
-					(reference "U5")
+					(reference "U6")
 					(unit 1)
 				)
@@
 		(dnp no)
 		(fields_autoplaced yes)
-		(property "Reference" "#PWR054"
+		(property "Reference" "#PWR059"
 			(at 148.59 184.15 0)
 			(effects
@@
 			(project "RamanSpectrometerBoard"
 				(path "/ab487c59-f066-48f5-a383-99e8eaf806bf/2495d964-2266-4066-961c-06fbcb7a3cda"
-					(reference "#PWR054")
+					(reference "#PWR059")
 					(unit 1)
 				)
@@
 		(dnp no)
 		(fields_autoplaced yes)
-		(property "Reference" "#PWR047"
+		(property "Reference" "#PWR052"
 			(at 63.5 184.15 0)
 			(effects
@@
 			(project "RamanSpectrometerBoard"
 				(path "/ab487c59-f066-48f5-a383-99e8eaf806bf/2495d964-2266-4066-961c-06fbcb7a3cda"
-					(reference "#PWR047")
+					(reference "#PWR052")
 					(unit 1)
 				)
@@
 		(dnp no)
 		(fields_autoplaced yes)
-		(property "Reference" "#PWR058"
+		(property "Reference" "#PWR063"
 			(at 193.04 35.56 0)
 			(effects
@@
 			(project "RamanSpectrometerBoard"
 				(path "/ab487c59-f066-48f5-a383-99e8eaf806bf/2495d964-2266-4066-961c-06fbcb7a3cda"
-					(reference "#PWR058")
+					(reference "#PWR063")
 					(unit 1)
 				)
@@
 		(dnp no)
 		(fields_autoplaced yes)
-		(property "Reference" "SW3"
+		(property "Reference" "SW2"
 			(at 139.7 167.64 0)
 			(effects
@@
 			(project "RamanSpectrometerBoard"
 				(path "/ab487c59-f066-48f5-a383-99e8eaf806bf/2495d964-2266-4066-961c-06fbcb7a3cda"
-					(reference "SW3")
+					(reference "SW2")
 					(unit 1)
 				)
@@
 		(on_board yes)
 		(dnp no)
-		(property "Reference" "C17"
+		(property "Reference" "C19"
 			(at 205.232 58.674 0)
 			(effects
@@
 			(project "RamanSpectrometerBoard"
 				(path "/ab487c59-f066-48f5-a383-99e8eaf806bf/2495d964-2266-4066-961c-06fbcb7a3cda"
-					(reference "C17")
+					(reference "C19")
 					(unit 1)
 				)
@@
 		(dnp no)
 		(fields_autoplaced yes)
-		(property "Reference" "#PWR056"
+		(property "Reference" "#PWR061"
 			(at 187.96 35.56 0)
 			(effects
@@
 			(project "RamanSpectrometerBoard"
 				(path "/ab487c59-f066-48f5-a383-99e8eaf806bf/2495d964-2266-4066-961c-06fbcb7a3cda"
-					(reference "#PWR056")
-					(unit 1)
-				)
+					(reference "#PWR061")
+					(unit 1)
+				)

Commit message: Finished laser diode layout
Parts:
- renumbered C14 to C15, C15 to C16, C16 to C17, C17 to C18, C18 to C19, C19 to C20
Changed lines of the file:
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@@
 		(dnp no)
 		(fields_autoplaced yes)
-		(property "Reference" "#PWR056"
+		(property "Reference" "#PWR058"
 			(at 86.36 35.56 0)
 			(effects
@@
 			(project "RamanSpectrometerBoard"
 				(path "/ab487c59-f066-48f5-a383-99e8eaf806bf/2495d964-2266-4066-961c-06fbcb7a3cda"
-					(reference "#PWR056")
+					(reference "#PWR058")
 					(unit 1)
 				)
@@
 		(dnp no)
 		(fields_autoplaced yes)
-		(property "Reference" "#PWR062"
+		(property "Reference" "#PWR064"
 			(at 190.5 87.63 0)
 			(effects
@@
 			(project "RamanSpectrometerBoard"
 				(path "/ab487c59-f066-48f5-a383-99e8eaf806bf/2495d964-2266-4066-961c-06fbcb7a3cda"
-					(reference "#PWR062")
+					(reference "#PWR064")
 					(unit 1)
 				)
@@
 		(on_board yes)
 		(dnp no)
-		(property "Reference" "C16"
+		(property "Reference" "C17"
 			(at 98.552 58.674 0)
 			(effects
@@
 			(project "RamanSpectrometerBoard"
 				(path "/ab487c59-f066-48f5-a383-99e8eaf806bf/2495d964-2266-4066-961c-06fbcb7a3cda"
-					(reference "C16")
+					(reference "C17")
 					(unit 1)
 				)
@@
 		(on_board yes)
 		(dnp no)
-		(property "Reference" "C14"
+		(property "Reference" "C15"
 			(at 67.818 41.91 0)
 			(effects
@@
 			(project "RamanSpectrometerBoard"
 				(path "/ab487c59-f066-48f5-a383-99e8eaf806bf/2495d964-2266-4066-961c-06fbcb7a3cda"
-					(reference "C14")
+					(reference "C15")
 					(unit 1)
 				)
@@
 		(dnp no)
 		(fields_autoplaced yes)
-		(property "Reference" "#PWR054"
+		(property "Reference" "#PWR056"
 			(at 81.28 35.56 0)
 			(effects
@@
 			(project "RamanSpectrometerBoard"
 				(path "/ab487c59-f066-48f5-a383-99e8eaf806bf/2495d964-2266-4066-961c-06fbcb7a3cda"
-					(reference "#PWR054")
+					(reference "#PWR056")
 					(unit 1)
 				)
@@
 		(on_board yes)
 		(dnp no)
-		(property "Reference" "#PWR065"
+		(property "Reference" "#PWR067"
 			(at 208.28 73.66 0)
 			(effects
@@
 			(project "RamanSpectrometerBoard"
 				(path "/ab487c59-f066-48f5-a383-99e8eaf806bf/2495d964-2266-4066-961c-06fbcb7a3cda"
-					(reference "#PWR065")
+					(reference "#PWR067")
 					(unit 1)
 				)
@@
 		(dnp no)
 		(fields_autoplaced yes)
-		(property "Reference" "#PWR055"
+		(property "Reference" "#PWR057"
 			(at 83.82 87.63 0)
 			(effects
@@
 			(project "RamanSpectrometerBoard"
 				(path "/ab487c59-f066-48f5-a383-99e8eaf806bf/2495d964-2266-4066-961c-06fbcb7a3cda"
-					(reference "#PWR055")
+					(reference "#PWR057")
 					(unit 1)
 				)
@@
 		(on_board yes)
 		(dnp no)
-		(property "Reference" "#PWR053"
+		(property "Reference" "#PWR055"
 			(at 76.2 54.61 0)
 			(effects
@@
 			(project "RamanSpectrometerBoard"
 				(path "/ab487c59-f066-48f5-a383-99e8eaf806bf/2495d964-2266-4066-961c-06fbcb7a3cda"
-					(reference "#PWR053")
+					(reference "#PWR055")
 					(unit 1)
 				)
@@
 		(on_board yes)
 		(dnp no)
-		(property "Reference" "#PWR060"
+		(property "Reference" "#PWR062"
 			(at 182.88 54.61 0)
 			(effects
@@
 			(project "RamanSpectrometerBoard"
 				(path "/ab487c59-f066-48f5-a383-99e8eaf806bf/2495d964-2266-4066-961c-06fbcb7a3cda"
-					(reference "#PWR060")
+					(reference "#PWR062")
 					(unit 1)
 				)
@@
 		(on_board yes)
 		(dnp no)
-		(property "Reference" "#PWR064"
+		(property "Reference" "#PWR066"
 			(at 198.12 54.61 0)
 			(effects
@@
 			(project "RamanSpectrometerBoard"
 				(path "/ab487c59-f066-48f5-a383-99e8eaf806bf/2495d964-2266-4066-961c-06fbcb7a3cda"
-					(reference "#PWR064")
+					(reference "#PWR066")
 					(unit 1)
 				)
@@
 		(dnp no)
 		(fields_autoplaced yes)
-		(property "Reference" "C15"
+		(property "Reference" "C16"
 			(at 95.25 41.9099 0)
 			(effects
@@
 			(project "RamanSpectrometerBoard"
 				(path "/ab487c59-f066-48f5-a383-99e8eaf806bf/2495d964-2266-4066-961c-06fbcb7a3cda"
-					(reference "C15")
+					(reference "C16")
 					(unit 1)
 				)
@@
 		(on_board yes)
 		(dnp no)
-		(property "Reference" "#PWR057"
+		(property "Reference" "#PWR059"
 			(at 91.44 54.61 0)
 			(effects
@@
 			(project "RamanSpectrometerBoard"
 				(path "/ab487c59-f066-48f5-a383-99e8eaf806bf/2495d964-2266-4066-961c-06fbcb7a3cda"
-					(reference "#PWR057")
+					(reference "#PWR059")
 					(unit 1)
 				)
@@
 		(on_board yes)
 		(dnp no)
-		(property "Reference" "#PWR058"
+		(property "Reference" "#PWR060"
 			(at 101.6 73.66 0)
 			(effects
@@
 			(project "RamanSpectrometerBoard"
 				(path "/ab487c59-f066-48f5-a383-99e8eaf806bf/2495d964-2266-4066-961c-06fbcb7a3cda"
-					(reference "#PWR058")
+					(reference "#PWR060")
 					(unit 1)
 				)
@@
 		(dnp no)
 		(fields_autoplaced yes)
-		(property "Reference" "C18"
+		(property "Reference" "C19"
 			(at 201.93 41.9099 0)
 			(effects
@@
 			(project "RamanSpectrometerBoard"
 				(path "/ab487c59-f066-48f5-a383-99e8eaf806bf/2495d964-2266-4066-961c-06fbcb7a3cda"
-					(reference "C18")
+					(reference "C19")
 					(unit 1)
 				)
@@
 		(on_board yes)
 		(dnp no)
-		(property "Reference" "C17"
+		(property "Reference" "C18"
 			(at 174.498 41.91 0)
 			(effects
@@
 			(project "RamanSpectrometerBoard"
 				(path "/ab487c59-f066-48f5-a383-99e8eaf806bf/2495d964-2266-4066-961c-06fbcb7a3cda"
-					(reference "C17")
+					(reference "C18")
 					(unit 1)
 				)
@@
 		(dnp no)
 		(fields_autoplaced yes)
-		(property "Reference" "#PWR059"
+		(property "Reference" "#PWR061"
 			(at 148.59 184.15 0)
 			(effects
@@
 			(project "RamanSpectrometerBoard"
 				(path "/ab487c59-f066-48f5-a383-99e8eaf806bf/2495d964-2266-4066-961c-06fbcb7a3cda"
-					(reference "#PWR059")
+					(reference "#PWR061")
 					(unit 1)
 				)
@@
 		(dnp no)
 		(fields_autoplaced yes)
-		(property "Reference" "#PWR052"
+		(property "Reference" "#PWR054"
 			(at 63.5 184.15 0)
 			(effects
@@
 			(project "RamanSpectrometerBoard"
 				(path "/ab487c59-f066-48f5-a383-99e8eaf806bf/2495d964-2266-4066-961c-06fbcb7a3cda"
-					(reference "#PWR052")
+					(reference "#PWR054")
 					(unit 1)
 				)
@@
 		(dnp no)
 		(fields_autoplaced yes)
-		(property "Reference" "#PWR063"
+		(property "Reference" "#PWR065"
 			(at 193.04 35.56 0)
 			(effects
@@
 			(project "RamanSpectrometerBoard"
 				(path "/ab487c59-f066-48f5-a383-99e8eaf806bf/2495d964-2266-4066-961c-06fbcb7a3cda"
-					(reference "#PWR063")
+					(reference "#PWR065")
 					(unit 1)
 				)
@@
 		(on_board yes)
 		(dnp no)
-		(property "Reference" "C19"
+		(property "Reference" "C20"
 			(at 205.232 58.674 0)
 			(effects
@@
 			(project "RamanSpectrometerBoard"
 				(path "/ab487c59-f066-48f5-a383-99e8eaf806bf/2495d964-2266-4066-961c-06fbcb7a3cda"
-					(reference "C19")
+					(reference "C20")
 					(unit 1)
 				)
@@
 		(dnp no)
 		(fields_autoplaced yes)
-		(property "Reference" "#PWR061"
+		(property "Reference" "#PWR063"
 			(at 187.96 35.56 0)
 			(effects
@@
 			(project "RamanSpectrometerBoard"
 				(path "/ab487c59-f066-48f5-a383-99e8eaf806bf/2495d964-2266-4066-961c-06fbcb7a3cda"
-					(reference "#PWR061")
-					(unit 1)
-				)
+					(reference "#PWR063")
+					(unit 1)
+				)
