File: Raman Spectrometer Board/LD_Buck.kicad_sch (KiCad schematic)
At the start: 10 parts, among them Q5 DMP3099L, U7 MAX1626ESA+T

Commit message: Began re-laying out laser driver section
Parts:
- renumbered C8 to C10, C8 to C11, C9 to C12, C10 to C13, D5 to D6, L2 to L1, Q5 to Q7, R12 to R23, R12 to R24, U7 to U5
Changed lines of the file:
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@@
 		(on_board yes)
 		(dnp no)
-		(property "Reference" "C8"
+		(property "Reference" "C10"
 			(at 60.96 40.0049 0)
 			(effects
@@
 			(project "RamanSpectrometerBoard"
 				(path "/ab487c59-f066-48f5-a383-99e8eaf806bf/42b2f347-68eb-4414-b5a4-00ef2fdb0e78"
-					(reference "C8")
+					(reference "C10")
 					(unit 1)
 				)
@@
 		(on_board yes)
 		(dnp no)
-		(property "Reference" "#PWR033"
+		(property "Reference" "#PWR046"
 			(at 64.77 78.74 0)
 			(effects
@@
 			(project "RamanSpectrometerBoard"
 				(path "/ab487c59-f066-48f5-a383-99e8eaf806bf/42b2f347-68eb-4414-b5a4-00ef2fdb0e78"
-					(reference "#PWR033")
+					(reference "#PWR046")
 					(unit 1)
 				)
@@
 		(dnp no)
 		(fields_autoplaced yes)
-		(property "Reference" "#PWR031"
+		(property "Reference" "#PWR044"
 			(at 64.77 34.29 0)
 			(effects
@@
 			(project "RamanSpectrometerBoard"
 				(path "/ab487c59-f066-48f5-a383-99e8eaf806bf/42b2f347-68eb-4414-b5a4-00ef2fdb0e78"
-					(reference "#PWR031")
+					(reference "#PWR044")
 					(unit 1)
 				)
@@
 		(on_board yes)
 		(dnp no)
-		(property "Reference" "#PWR041"
+		(property "Reference" "#PWR051"
 			(at 156.21 91.44 0)
 			(effects
@@
 			(project "RamanSpectrometerBoard"
 				(path "/ab487c59-f066-48f5-a383-99e8eaf806bf/42b2f347-68eb-4414-b5a4-00ef2fdb0e78"
-					(reference "#PWR041")
+					(reference "#PWR051")
 					(unit 1)
 				)
@@
 		(dnp no)
 		(fields_autoplaced yes)
-		(property "Reference" "C10"
+		(property "Reference" "C13"
 			(at 160.02 78.1049 0)
 			(effects
@@
 			(project "RamanSpectrometerBoard"
 				(path "/ab487c59-f066-48f5-a383-99e8eaf806bf/42b2f347-68eb-4414-b5a4-00ef2fdb0e78"
-					(reference "C10")
+					(reference "C13")
 					(unit 1)
 				)
@@
 		(dnp no)
 		(fields_autoplaced yes)
-		(property "Reference" "R12"
+		(property "Reference" "R24"
 			(at 124.46 45.7199 0)
 			(effects
@@
 			(project "RamanSpectrometerBoard"
 				(path "/ab487c59-f066-48f5-a383-99e8eaf806bf/42b2f347-68eb-4414-b5a4-00ef2fdb0e78"
-					(reference "R12")
+					(reference "R24")
 					(unit 1)
 				)
@@
 		(on_board yes)
 		(dnp no)
-		(property "Reference" "C9"
+		(property "Reference" "C12"
 			(at 72.136 64.77 0)
 			(effects
@@
 			(project "RamanSpectrometerBoard"
 				(path "/ab487c59-f066-48f5-a383-99e8eaf806bf/42b2f347-68eb-4414-b5a4-00ef2fdb0e78"
-					(reference "C9")
+					(reference "C12")
 					(unit 1)
 				)
@@
 		(on_board yes)
 		(dnp no)
-		(property "Reference" "C8"
+		(property "Reference" "C11"
 			(at 72.136 40.64 0)
 			(effects
@@
 			(project "RamanSpectrometerBoard"
 				(path "/ab487c59-f066-48f5-a383-99e8eaf806bf/42b2f347-68eb-4414-b5a4-00ef2fdb0e78"
-					(reference "C8")
+					(reference "C11")
 					(unit 1)
 				)
@@
 		(on_board yes)
 		(dnp no)
-		(property "Reference" "Q5"
+		(property "Reference" "Q7"
 			(at 125.73 62.2301 0)
 			(effects
@@
 			(project "RamanSpectrometerBoard"
 				(path "/ab487c59-f066-48f5-a383-99e8eaf806bf/42b2f347-68eb-4414-b5a4-00ef2fdb0e78"
-					(reference "Q5")
+					(reference "Q7")
 					(unit 1)
 				)
@@
 		(on_board yes)
 		(dnp no)
-		(property "Reference" "#PWR035"
+		(property "Reference" "#PWR048"
 			(at 83.82 78.74 0)
 			(effects
@@
 			(project "RamanSpectrometerBoard"
 				(path "/ab487c59-f066-48f5-a383-99e8eaf806bf/42b2f347-68eb-4414-b5a4-00ef2fdb0e78"
-					(reference "#PWR035")
+					(reference "#PWR048")
 					(unit 1)
 				)
@@
 		(on_board yes)
 		(dnp no)
-		(property "Reference" "D5"
+		(property "Reference" "D6"
 			(at 119.38 75.8824 90)
 			(effects
@@
 			(project "RamanSpectrometerBoard"
 				(path "/ab487c59-f066-48f5-a383-99e8eaf806bf/42b2f347-68eb-4414-b5a4-00ef2fdb0e78"
-					(reference "D5")
+					(reference "D6")
 					(unit 1)
 				)
@@
 		(on_board yes)
 		(dnp no)
-		(property "Reference" "L2"
+		(property "Reference" "L1"
 			(at 138.43 66.294 90)
 			(effects
@@
 			(project "RamanSpectrometerBoard"
 				(path "/ab487c59-f066-48f5-a383-99e8eaf806bf/42b2f347-68eb-4414-b5a4-00ef2fdb0e78"
-					(reference "L2")
+					(reference "L1")
 					(unit 1)
 				)
@@
 		(on_board yes)
 		(dnp no)
-		(property "Reference" "#PWR032"
+		(property "Reference" "#PWR045"
 			(at 64.77 53.34 0)
 			(effects
@@
 			(project "RamanSpectrometerBoard"
 				(path "/ab487c59-f066-48f5-a383-99e8eaf806bf/42b2f347-68eb-4414-b5a4-00ef2fdb0e78"
-					(reference "#PWR032")
+					(reference "#PWR045")
 					(unit 1)
 				)
@@
 		(on_board yes)
 		(dnp no)
-		(property "Reference" "R12"
+		(property "Reference" "R23"
 			(at 62.23 64.7699 0)
 			(effects
@@
 			(project "RamanSpectrometerBoard"
 				(path "/ab487c59-f066-48f5-a383-99e8eaf806bf/42b2f347-68eb-4414-b5a4-00ef2fdb0e78"
-					(reference "R12")
+					(reference "R23")
 					(unit 1)
 				)
@@
 		(on_board yes)
 		(dnp no)
-		(property "Reference" "#PWR039"
+		(property "Reference" "#PWR049"
 			(at 121.92 90.17 0)
 			(effects
@@
 			(project "RamanSpectrometerBoard"
 				(path "/ab487c59-f066-48f5-a383-99e8eaf806bf/42b2f347-68eb-4414-b5a4-00ef2fdb0e78"
-					(reference "#PWR039")
+					(reference "#PWR049")
 					(unit 1)
 				)
@@
 		(on_board yes)
 		(dnp no)
-		(property "Reference" "#PWR034"
+		(property "Reference" "#PWR047"
 			(at 77.47 53.34 0)
 			(effects
@@
 			(project "RamanSpectrometerBoard"
 				(path "/ab487c59-f066-48f5-a383-99e8eaf806bf/42b2f347-68eb-4414-b5a4-00ef2fdb0e78"
-					(reference "#PWR034")
+					(reference "#PWR047")
 					(unit 1)
 				)
@@
 		(on_board yes)
 		(dnp no)
-		(property "Reference" "#PWR040"
+		(property "Reference" "#PWR050"
 			(at 156.21 68.58 0)
 			(effects
@@
 			(project "RamanSpectrometerBoard"
 				(path "/ab487c59-f066-48f5-a383-99e8eaf806bf/42b2f347-68eb-4414-b5a4-00ef2fdb0e78"
-					(reference "#PWR040")
+					(reference "#PWR050")
 					(unit 1)
 				)
@@
 		(dnp no)
 		(fields_autoplaced yes)
-		(property "Reference" "U7"
+		(property "Reference" "U5"
 			(at 93.98 45.72 0)
 			(effects
@@
 			(project "RamanSpectrometerBoard"
 				(path "/ab487c59-f066-48f5-a383-99e8eaf806bf/42b2f347-68eb-4414-b5a4-00ef2fdb0e78"
-					(reference "U7")
-					(unit 1)
-				)
+					(reference "U5")
+					(unit 1)
+				)

Commit message: Finished laser diode layout
Parts:
- renumbered C10 to C11, C11 to C12, C12 to C13, C13 to C14
Changed lines of the file:
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@@
 		(on_board yes)
 		(dnp no)
-		(property "Reference" "C10"
+		(property "Reference" "C11"
 			(at 60.96 40.0049 0)
 			(effects
@@
 			(project "RamanSpectrometerBoard"
 				(path "/ab487c59-f066-48f5-a383-99e8eaf806bf/42b2f347-68eb-4414-b5a4-00ef2fdb0e78"
-					(reference "C10")
+					(reference "C11")
 					(unit 1)
 				)
@@
 		(on_board yes)
 		(dnp no)
-		(property "Reference" "#PWR046"
+		(property "Reference" "#PWR048"
 			(at 64.77 78.74 0)
 			(effects
@@
 			(project "RamanSpectrometerBoard"
 				(path "/ab487c59-f066-48f5-a383-99e8eaf806bf/42b2f347-68eb-4414-b5a4-00ef2fdb0e78"
-					(reference "#PWR046")
+					(reference "#PWR048")
 					(unit 1)
 				)
@@
 		(dnp no)
 		(fields_autoplaced yes)
-		(property "Reference" "#PWR044"
+		(property "Reference" "#PWR046"
 			(at 64.77 34.29 0)
 			(effects
@@
 			(project "RamanSpectrometerBoard"
 				(path "/ab487c59-f066-48f5-a383-99e8eaf806bf/42b2f347-68eb-4414-b5a4-00ef2fdb0e78"
-					(reference "#PWR044")
+					(reference "#PWR046")
 					(unit 1)
 				)
@@
 		(on_board yes)
 		(dnp no)
-		(property "Reference" "#PWR051"
+		(property "Reference" "#PWR053"
 			(at 156.21 91.44 0)
 			(effects
@@
 			(project "RamanSpectrometerBoard"
 				(path "/ab487c59-f066-48f5-a383-99e8eaf806bf/42b2f347-68eb-4414-b5a4-00ef2fdb0e78"
-					(reference "#PWR051")
+					(reference "#PWR053")
 					(unit 1)
 				)
@@
 		(dnp no)
 		(fields_autoplaced yes)
-		(property "Reference" "C13"
+		(property "Reference" "C14"
 			(at 160.02 78.1049 0)
 			(effects
@@
 			(project "RamanSpectrometerBoard"
 				(path "/ab487c59-f066-48f5-a383-99e8eaf806bf/42b2f347-68eb-4414-b5a4-00ef2fdb0e78"
-					(reference "C13")
+					(reference "C14")
 					(unit 1)
 				)
@@
 		(on_board yes)
 		(dnp no)
-		(property "Reference" "C12"
+		(property "Reference" "C13"
 			(at 72.136 64.77 0)
 			(effects
@@
 			(project "RamanSpectrometerBoard"
 				(path "/ab487c59-f066-48f5-a383-99e8eaf806bf/42b2f347-68eb-4414-b5a4-00ef2fdb0e78"
-					(reference "C12")
+					(reference "C13")
 					(unit 1)
 				)
@@
 		(on_board yes)
 		(dnp no)
-		(property "Reference" "C11"
+		(property "Reference" "C12"
 			(at 72.136 40.64 0)
 			(effects
@@
 			(project "RamanSpectrometerBoard"
 				(path "/ab487c59-f066-48f5-a383-99e8eaf806bf/42b2f347-68eb-4414-b5a4-00ef2fdb0e78"
-					(reference "C11")
+					(reference "C12")
 					(unit 1)
 				)
@@
 		(on_board yes)
 		(dnp no)
-		(property "Reference" "#PWR048"
+		(property "Reference" "#PWR050"
 			(at 83.82 78.74 0)
 			(effects
@@
 			(project "RamanSpectrometerBoard"
 				(path "/ab487c59-f066-48f5-a383-99e8eaf806bf/42b2f347-68eb-4414-b5a4-00ef2fdb0e78"
-					(reference "#PWR048")
+					(reference "#PWR050")
 					(unit 1)
 				)
@@
 		(on_board yes)
 		(dnp no)
-		(property "Reference" "#PWR045"
+		(property "Reference" "#PWR047"
 			(at 64.77 53.34 0)
 			(effects
@@
 			(project "RamanSpectrometerBoard"
 				(path "/ab487c59-f066-48f5-a383-99e8eaf806bf/42b2f347-68eb-4414-b5a4-00ef2fdb0e78"
-					(reference "#PWR045")
+					(reference "#PWR047")
 					(unit 1)
 				)
@@
 		(on_board yes)
 		(dnp no)
-		(property "Reference" "#PWR049"
+		(property "Reference" "#PWR051"
 			(at 121.92 90.17 0)
 			(effects
@@
 			(project "RamanSpectrometerBoard"
 				(path "/ab487c59-f066-48f5-a383-99e8eaf806bf/42b2f347-68eb-4414-b5a4-00ef2fdb0e78"
-					(reference "#PWR049")
+					(reference "#PWR051")
 					(unit 1)
 				)
@@
 		(on_board yes)
 		(dnp no)
-		(property "Reference" "#PWR047"
+		(property "Reference" "#PWR049"
 			(at 77.47 53.34 0)
 			(effects
@@
 			(project "RamanSpectrometerBoard"
 				(path "/ab487c59-f066-48f5-a383-99e8eaf806bf/42b2f347-68eb-4414-b5a4-00ef2fdb0e78"
-					(reference "#PWR047")
+					(reference "#PWR049")
 					(unit 1)
 				)
@@
 		(on_board yes)
 		(dnp no)
-		(property "Reference" "#PWR050"
+		(property "Reference" "#PWR052"
 			(at 156.21 68.58 0)
 			(effects
@@
 			(project "RamanSpectrometerBoard"
 				(path "/ab487c59-f066-48f5-a383-99e8eaf806bf/42b2f347-68eb-4414-b5a4-00ef2fdb0e78"
-					(reference "#PWR050")
-					(unit 1)
-				)
+					(reference "#PWR052")
+					(unit 1)
+				)

Commit message: Laser switch
Parts:
- added C19, C20: 10uF, Capacitor_SMD:C_0603_1608Metric_Pad1.08x0.95mm_HandSolder, symbol Device:C
- added Q8: BSS138, Package_TO_SOT_SMD:SOT-23, symbol Transistor_FET:BSS138
- added R29: 100, Resistor_SMD:R_0603_1608Metric, symbol Device:R_US
- added R30: 100k, Resistor_SMD:R_0603_1608Metric, symbol Device:R_US
- added U8: OKI, Converter_DCDC:Converter_DCDC_Murata_OKI-78SR_Vertical, symbol MRDT_Devices:OKI
Connections:
- net +12V: now also C19.1, R30.1, U8.1 (Vi)
- net +3.3V_{LD}: now also C20.1, U8.3 (Vo)
- net GND: now also C19.2, C20.2, Q8.2 (S), U8.2 (GND)
- net at R23.1: now also Q8.1 (G), R29.2; no longer U5.3 (SHDN)
- new net: Q8.3 (D), R30.2, U5.3 (SHDN)
- new net SHDN: R29.1
Other:
- note added: "OKI"
- moved on the sheet: R23

Commit message: Laser driver capacitor
Parts:
- removed C11: 100 µF, LaserDriverRev2Library:CAPMP6.3X3.2_2.8N_KEM, symbol Device:C_Polarized_US
- added C11, C21: 47uF, Capacitor_SMD:C_0603_1608Metric, symbol Device:C
Connections:
- net +12V: now also C11.1, C21.1
- net GND: now also C11.2, C21.2
Changed lines of the file:
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@@
+	)
+	(junction
+		(at 64.77 45.72)
+		(diameter 0)
+		(color 0 0 0 0)
 	)
 	(junction
@@
 	(wire
 		(pts
-			(xy 64.77 46.99) (xy 64.77 45.72)
-		)
-		(stroke
-			(width 0)
-			(type default)
-		)
-	)
-	(wire
-		(pts
 			(xy 38.1 109.22) (xy 54.61 109.22)
 		)
@@
 	(wire
 		(pts
+			(xy 54.61 38.1) (xy 54.61 34.29)
+		)
+		(stroke
+			(width 0)
+			(type default)
+		)
+	)
+	(wire
+		(pts
 			(xy 121.92 34.29) (xy 121.92 43.18)
 		)
@@
 	(wire
 		(pts
+			(xy 54.61 34.29) (xy 64.77 34.29)
+		)
+		(stroke
+			(width 0)
+			(type default)
+		)
+	)
+	(wire
+		(pts
 			(xy 33.02 59.69) (xy 33.02 64.77)
 		)
@@
 	(wire
 		(pts
+			(xy 64.77 45.72) (xy 64.77 46.99)
+		)
+		(stroke
+			(width 0)
+			(type default)
+		)
+	)
+	(wire
+		(pts
 			(xy 44.45 52.07) (xy 44.45 54.61)
 		)
@@
 		(pts
 			(xy 64.77 30.48) (xy 64.77 34.29)
+		)
+		(stroke
+			(width 0)
+			(type default)
+		)
+	)
+	(wire
+		(pts
+			(xy 54.61 45.72) (xy 64.77 45.72)
 		)
 		(stroke
@@
 	)
 	(symbol
-		(lib_id "Device:C_Polarized_US")
-		(at 64.77 41.91 0)
-		(mirror y)
-		(unit 1)
-		(exclude_from_sim no)
-		(in_bom yes)
-		(on_board yes)
-		(dnp no)
-		(property "Reference" "C11"
-			(at 60.96 40.0049 0)
-			(effects
-				(font
-					(size 1.27 1.27)
-				)
-				(justify left)
-			)
-		)
-		(property "Value" "100 µF"
-			(at 60.96 42.5449 0)
-			(effects
-				(font
-					(size 1.27 1.27)
-				)
-				(justify left)
-			)
-		)
-		(property "Footprint" "LaserDriverRev2Library:CAPMP6.3X3.2_2.8N_KEM"
-			(at 64.77 41.91 0)
-			(effects
-				(font
-					(size 1.27 1.27)
-				)
-				(hide yes)
-			)
-		)
-		(property "Datasheet" "https://www.digikey.com/en/products/detail/kemet/T495C107K006ATE075/1829938"
-			(at 64.77 41.91 0)
-			(effects
-				(font
-					(size 1.27 1.27)
-				)
-				(hide yes)
-			)
-		)
-		(property "Description" "100 µF Molded Tantalum Capacitors 6.3 V 2312 (6032 Metric) 75mOhm"
-			(at 64.77 41.91 0)
-			(effects
-				(font
-					(size 1.27 1.27)
-				)
-				(hide yes)
-			)
-		)
-		(pin "2"
-		)
-		(pin "1"
-		)
-		(instances
-			(project "RamanSpectrometerBoard"
-				(path "/ab487c59-f066-48f5-a383-99e8eaf806bf/42b2f347-68eb-4414-b5a4-00ef2fdb0e78"
-					(reference "C11")
-					(unit 1)
-				)
-			)
-		)
-	)
-	(symbol
 		(lib_id "power:GND")
 		(at 33.02 74.93 0)
@@
 	(symbol
 		(lib_id "Device:C")
+		(at 64.77 41.91 0)
+		(mirror y)
+		(unit 1)
+		(exclude_from_sim no)
+		(in_bom yes)
+		(on_board yes)
+		(dnp no)
+		(property "Reference" "C11"
+			(at 59.436 40.64 0)
+			(effects
+				(font
+					(size 1.27 1.27)
+				)
+			)
+		)
+		(property "Value" "47uF"
+			(at 59.436 42.926 0)
+			(effects
+				(font
+					(size 1.27 1.27)
+				)
+			)
+		)
+		(property "Footprint" "Capacitor_SMD:C_0603_1608Metric"
+			(at 63.8048 45.72 0)
+			(effects
+				(font
+					(size 1.27 1.27)
+				)
+				(hide yes)
+			)
+		)
+		(property "Datasheet" "(Standards)"
+			(at 64.77 41.91 0)
+			(effects
+				(font
+					(size 1.27 1.27)
+				)
+				(hide yes)
+			)
+		)
+		(property "Description" "0.47uF, 0603"
+			(at 64.77 41.91 0)
+			(effects
+				(font
+					(size 1.27 1.27)
+				)
+				(hide yes)
+			)
+		)
+		(pin "1"
+		)
+		(pin "2"
+		)
+		(instances
+			(project "RamanSpectrometerBoard"
+				(path "/ab487c59-f066-48f5-a383-99e8eaf806bf/42b2f347-68eb-4414-b5a4-00ef2fdb0e78"
+					(reference "C11")
+					(unit 1)
+				)
+			)
+		)
+	)
+	(symbol
+		(lib_id "Device:C")
 		(at 71.12 104.14 0)
 		(unit 1)
@@
 					(unit 1)
 				)
+			)
+		)
+	)
+	(symbol
+		(lib_id "Device:C")
+		(at 54.61 41.91 0)
+		(mirror y)
+		(unit 1)
+		(exclude_from_sim no)
+		(in_bom yes)
+		(on_board yes)
+		(dnp no)
+		(property "Reference" "C21"
+			(at 49.276 40.64 0)
+			(effects
+				(font
+					(size 1.27 1.27)
+				)
+			)
+		)
+		(property "Value" "47uF"
+			(at 49.276 42.926 0)
+			(effects
+				(font
+					(size 1.27 1.27)
+				)
+			)
+		)
+		(property "Footprint" "Capacitor_SMD:C_0603_1608Metric"
+			(at 53.6448 45.72 0)
+			(effects
+				(font
+					(size 1.27 1.27)
+				)
+				(hide yes)
+			)
+		)
+		(property "Datasheet" "(Standards)"
+			(at 54.61 41.91 0)
+			(effects
+				(font
+					(size 1.27 1.27)
+				)
+				(hide yes)
+			)
+		)
+		(property "Description" "0.47uF, 0603"
+			(at 54.61 41.91 0)
+			(effects
+				(font
+					(size 1.27 1.27)
+				)
+				(hide yes)
+			)
+		)
+		(pin "1"
+		)
+		(pin "2"
+		)
+		(instances
+			(project "RamanSpectrometerBoard"
+				(path "/ab487c59-f066-48f5-a383-99e8eaf806bf/42b2f347-68eb-4414-b5a4-00ef2fdb0e78"
+					(reference "C21")
+					(unit 1)
+				)

Commit message: Post review laser driver edits
Other:
- moved on the sheet: C12, C21
