File: CCD Breakout/CCD_Breakout/CCD_Breakout/adc.kicad_sch (KiCad schematic)
At the start: 8 parts, among them U3 ADC-MCP33151

Commit message: Added 3.3v to ADC
Connections:
- net +5V: no longer C4.1, U3.1 (VREF)
- new net +3V3: C4.1, U3.1 (VREF)
Changed lines of the file:
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@@
 	)
 	(junction
-		(at 121.92 58.42)
+		(at 129.54 63.5)
 		(diameter 0)
 		(color 0 0 0 0)
@@
 	)
 	(junction
-		(at 129.54 63.5)
-		(diameter 0)
-		(color 0 0 0 0)
-	)
-	(junction
 		(at 121.92 91.44)
 		(diameter 0)
@@
 	(wire
 		(pts
-			(xy 129.54 63.5) (xy 129.54 58.42)
-		)
-		(stroke
-			(width 0)
-			(type default)
-		)
-	)
-	(wire
-		(pts
 			(xy 154.94 76.2) (xy 154.94 77.47)
 		)
@@
 	(wire
 		(pts
+			(xy 129.54 55.88) (xy 129.54 63.5)
+		)
+		(stroke
+			(width 0)
+			(type default)
+		)
+	)
+	(wire
+		(pts
 			(xy 129.54 86.36) (xy 129.54 63.5)
 		)
@@
 		(pts
 			(xy 78.74 81.28) (xy 97.79 81.28)
-		)
-		(stroke
-			(width 0)
-			(type default)
-		)
-	)
-	(wire
-		(pts
-			(xy 121.92 58.42) (xy 129.54 58.42)
 		)
 		(stroke
@@
 					(unit 1)
 				)
+			)
+		)
+	)
+	(symbol
+		(lib_id "power:+3V3")
+		(at 129.54 55.88 0)
+		(unit 1)
+		(exclude_from_sim no)
+		(in_bom yes)
+		(on_board yes)
+		(dnp no)
+		(fields_autoplaced yes)
+		(property "Reference" "#PWR026"
+			(at 129.54 59.69 0)
+			(effects
+				(font
+					(size 1.27 1.27)
+				)
+				(hide yes)
+			)
+		)
+		(property "Value" "+3V3"
+			(at 129.54 50.8 0)
+			(effects
+				(font
+					(size 1.27 1.27)
+				)
+			)
+		)
+		(property "Footprint" ""
+			(at 129.54 55.88 0)
+			(effects
+				(font
+					(size 1.27 1.27)
+				)
+				(hide yes)
+			)
+		)
+		(property "Datasheet" ""
+			(at 129.54 55.88 0)
+			(effects
+				(font
+					(size 1.27 1.27)
+				)
+				(hide yes)
+			)
+		)
+		(property "Description" "Power symbol creates a global label with name \"+3V3\""
+			(at 129.54 55.88 0)
+			(effects
+				(font
+					(size 1.27 1.27)
+				)
+				(hide yes)
+			)
+		)
+		(pin "1"
+		)
+		(instances
+			(project ""
+				(path "/102965ac-29c6-4f96-94a4-d07431f6d693/a53142f3-0354-4e7c-bbfe-f09d56efc2e2"
+					(reference "#PWR026")
+					(unit 1)
+				)

Commit message: zener diode
Parts:
- D1: value CMDZ1L8 -> BZX8850S-B1V8-QYL
Changed lines of the file:
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@@
 			)
 		)
-		(property "Value" "CMDZ1L8"
+		(property "Value" "BZX8850S-B1V8-QYL"
 			(at 64.77 77.4699 90)
 			(effects
@@
 			)
 		)
-		(property "Datasheet" "https://my.centralsemi.com/datasheets/CMDZ5L1-36L.PDF"
+		(property "Datasheet" "https://assets.nexperia.com/documents/data-sheet/BZX8450-Q_SER.pdf"
 			(at 62.23 76.2 0)
 			(effects

Commit message: Draft layout design
Parts:
- D1: value BZX8850S-B1V8-QYL -> CMDZ1L8
- R7: value 100 -> 15
Changed lines of the file:
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@@
 			)
 		)
-		(property "Value" "100"
+		(property "Value" "15"
 			(at 114.3 96.774 90)
 			(effects
@@
 			)
 		)
-		(property "Value" "BZX8850S-B1V8-QYL"
+		(property "Value" "CMDZ1L8"
 			(at 64.77 77.4699 90)
 			(effects
@@
 			)
 		)
-		(property "Datasheet" "https://assets.nexperia.com/documents/data-sheet/BZX8450-Q_SER.pdf"
+		(property "Datasheet" "https://my.centralsemi.com/datasheets/CMDZ5L1-36L.PDF"
 			(at 62.23 76.2 0)
 			(effects

Commit message: Fix Layout Issues
Parts:
- U3: footprint (none) -> CCD:Untitled
Changed lines of the file:
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@@
 			)
 		)
-		(property "Footprint" ""
+		(property "Footprint" "CCD:Untitled"
 			(at 142.24 91.44 0)
 			(effects

Commit message: typos
Parts:
- C16: renamed from 2.2nF1; value C -> 2.2nF
- R2: value 1000 -> 1k
Changed lines of the file:
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@@
 			)
 		)
-		(property "Value" "1000"
+		(property "Value" "1k"
 			(at 64.77 63.4999 0)
 			(effects
@@
 		(on_board yes)
 		(dnp no)
-		(property "Reference" "2.2nF1"
+		(property "Reference" "C16"
 			(at 123.19 94.996 0)
 			(effects
@@
 			)
 		)
-		(property "Value" "C"
+		(property "Value" "2.2nF"
 			(at 123.19 97.536 0)
 			(effects
@@
 			(project ""
 				(path "/102965ac-29c6-4f96-94a4-d07431f6d693/a53142f3-0354-4e7c-bbfe-f09d56efc2e2"
-					(reference "2.2nF1")
-					(unit 1)
-				)
+					(reference "C16")
+					(unit 1)
+				)

Commit message: CRD Issues
Parts:
- C4: footprint Capacitor_Tantalum_SMD:CP_EIA-1608-08_AVX-J_HandSolder -> Capacitor_Tantalum_SMD:CP_EIA-2012-12_Kemet-R_HandSolder
- D1: footprint Diode_THT:D_DO-41_SOD81_P10.16mm_Horizontal -> Diode_SMD:D_SOD-323_HandSoldering
Changed lines of the file:
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@@
 			)
 		)
-		(property "Footprint" "Diode_THT:D_DO-41_SOD81_P10.16mm_Horizontal"
+		(property "Footprint" "Diode_SMD:D_SOD-323_HandSoldering"
 			(at 57.785 76.2 0)
 			(effects
@@
 			)
 		)
-		(property "Footprint" "Capacitor_Tantalum_SMD:CP_EIA-1608-08_AVX-J_HandSolder"
+		(property "Footprint" "Capacitor_Tantalum_SMD:CP_EIA-2012-12_Kemet-R_HandSolder"
 			(at 135.89 68.58 0)
 			(effects

Commit message: Fix CDR
Changed lines of the file:
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@@
+		)
+	)
+	(text_box "ADC"
+		(exclude_from_sim no)
+		(at 48.26 43.18 0)
+		(size 132.08 76.2)
+		(margins 0.9525 0.9525 0.9525 0.9525)
+		(stroke
+			(width 0)
+			(type solid)
+		)
+		(fill
+			(type none)
+		)
+		(effects
+			(font
+				(size 1.27 1.27)
+			)
+			(justify left top)
 		)
 	)
