File: CCD Breakout/CCD_Breakout/CCD_Breakout/CCD_BreakoutRev1.kicad_pcb (KiCad board)
At the start: 2 copper layers, 68.8 x 25.4 mm, 47 parts, among them Q1 SI01P10-TP, Q2 SI01P10-TP, U1 CCD, U3 ADC-MCP33151, U5 74HC541PW_118, U8 OPA4322AIPWR

Commit message: Rev2 Push
Parts:
- added 1V8: 1V8, TestPoint:TestPoint_Pad_D1.5mm, F.Cu at (153.9, 109.6)
- added 3V3: 3V3, TestPoint:TestPoint_Pad_D1.5mm, F.Cu at (156.6, 109.6)
- added 5V: 5V, TestPoint:TestPoint_Pad_D1.5mm, F.Cu at (126.1, 95.4)
- added AIN+: AIN+, TestPoint:TestPoint_Pad_D1.5mm, B.Cu at (149.1, 106.7)
- added D1: CMDZ1L8, Diode_SMD:D_SOD-323_HandSoldering, F.Cu at (163.6, 109.6)
- added R2: 1k, Resistor_SMD:R_0603_1608Metric_Pad0.98x0.95mm_HandSolder, F.Cu at (162.7, 107.0)
- added Video: Video, TestPoint:TestPoint_Pad_D1.5mm, F.Cu at (159.5, 109.6)
- TP3: value 5V -> 3V3
- moved C5 136.6 mm to (166.9, 103.9), turned to 0 degrees
- moved C4 120.8 mm to (147.4, 110.3), turned to 0 degrees
- moved R7 116.0 mm to (149.0, 108.5)
- moved C16 113.6 mm to (146.5, 107.5), turned to 90 degrees
- moved U3 112.5 mm to (142.8, 108.5), turned to 90 degrees
- moved C6 111.3 mm to (138.3, 109.5), turned to 180 degrees
- moved R15 106.2 mm to (167.8, 98.7), turned to -90 degrees
- moved R14 103.1 mm to (161.7, 103.6), turned to 180 degrees
- moved R11 101.0 mm to (128.1, 108.8)
- moved TP1 99.2 mm to (127.2, 55.8)
- moved R8 96.2 mm to (167.8, 95.2), turned to 90 degrees
- moved Q1 95.9 mm to (125.5, 109.0)
- moved TP4 94.7 mm to (127.2, 62.9)
- moved R4 91.1 mm to (150.8, 105.7)
- moved TP5 90.4 mm to (127.2, 66.4)
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Routing:
- net +5V: track 0.00 -> 118.0 mm, vias 0 -> 11
- net /ADC/SDI: track 40.8 -> 0.00 mm, vias 3 -> 0
- net /CCD/opINB+: track 0.00 -> 39.8 mm, vias 0 -> 5
- net /CCD/opINA+: track 0.00 -> 39.3 mm, vias 0 -> 4
- net +3V3: track 0.00 -> 39.1 mm, vias 0 -> 3
- net +1V8: track 0.00 -> 32.7 mm, vias 0 -> 3
- net unconnected-(U5-Y3-Pad15): track 0.00 -> 23.8 mm, vias 0 -> 1
- net /CCD/Trigb: track 0.00 -> 21.4 mm, vias 0 -> 2
- net /ADC/Video: track 0.00 -> 20.2 mm, vias 0 -> 2
- net /ADC/TRIG: track 41.8 -> 22.2 mm, vias 3 -> 2
- net /CCD/CLKb: track 0.00 -> 17.9 mm, vias 0 -> 2
- net /CCD/STb: track 0.00 -> 17.4 mm, vias 0 -> 4
- net /CCD/EOSb: track 0.00 -> 16.2 mm, vias 0 -> 2
- net Net-(Q2-S): track 0.00 -> 10.2 mm
- net /CCD/ST: track 15.1 -> 24.5 mm, vias 1 -> 3
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- added copper zone on F.Cu, net +5V
Other:
- board text added: "ADC"
- board text added: "Octal Buffer"
- board text added: "V Shifter"
