File: CCD Breakout/CCD_Breakout.kicad_pcb (KiCad board)
At the start: 2 copper layers, 68.8 x 25.4 mm, 47 parts, among them Q1 SI01P10-TP, Q2 SI01P10-TP, U1 CCD, U3 ADC-MCP33151, U5 74HC541PW_118, U8 OPA4322AIPWR

Commit message: Silkscreen Update
Parts:
- added G***: LOGO, Silkscreens:GVSigniture, F.Cu at (45.5, 89.2)
Other:
- board text added: "CMOS Board, Rev 2"
- board text added: "Mars Rover Design Team Missouri S&T"

Commit message: 3d Models added
Other:
- board text added: "+3V3"
- board text added: "+5V"
- board text added: "ADC_CLK"
- board text added: "CMOS_CLK"
- board text added: "GND"
- board text added: "OUT"
- board text added: "SDI"
- board text added: "ST"
- board text added: "Trig"
- board text added: "Trig_OUT"
Changed lines of the file:
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@@
 		)
 		(embedded_fonts no)
+		(model "D:/Desktop/Rover/Libraries/RamanSpectrometer_Hardware/lib/3d/OPA4322AIPWR.step"
+			(offset
+				(xyz 0 0 0)
+			)
+			(scale
+				(xyz 1 1 1)
+			)
+			(rotate
+				(xyz -90 -0 -0)
+			)
+		)
 	)
 	(footprint "Resistor_SMD:R_0603_1608Metric_Pad0.98x0.95mm_HandSolder"
@@
 			)
 		)
+		(model "D:/Desktop/Rover/Libraries/RamanSpectrometer_Hardware/lib/3d/SL_10.stp"
+			(offset
+				(xyz 11.43 0 8.255)
+			)
+			(scale
+				(xyz 1 1 1)
+			)
+			(rotate
+				(xyz -0 -0 -0)
+			)
+		)
 	)
 	(footprint "CCD:SOT-23_MCC-L"
@@
 		(tags "resistor handsolder")
 		(property "Reference" "R14"
-			(at -0.254 -1.651 90)
+			(at 2.032 0 180)
 			(layer "F.SilkS")
 			(effects
@@
 		)
 		(embedded_fonts no)
+		(model "D:/Desktop/Rover/Libraries/RamanSpectrometer_Hardware/lib/3d/74HC541PW_118.step"
+			(offset
+				(xyz 0 0 0)
+			)
+			(scale
+				(xyz 1 1 1)
+			)
+			(rotate
+				(xyz -90 -0 -0)
+			)
+		)
 	)
 	(footprint "Capacitor_SMD:C_0603_1608Metric_Pad1.08x0.95mm_HandSolder"
@@
 		)
 		(embedded_fonts no)
+		(model "D:/Desktop/Rover/Libraries/RamanSpectrometer_Hardware/lib/3d/MSOP10_MS_MCH.step"
+			(offset
+				(xyz 0 0 0)
+			)
+			(scale
+				(xyz 1 1 1)
+			)
+			(rotate
+				(xyz -0 -0 -90)
+			)
+		)
 	)
 	(footprint "Silkscreens:MST_Smaller"
@@
 		(layer "Edge.Cuts")
 	)
+	(gr_text "Trig\n"
+		(at 54.977224 66.0654 180)
+		(layer "F.SilkS")
+		(effects
+			(font
+				(size 0.5 0.5)
+				(thickness 0.125)
+				(bold yes)
+			)
+			(justify left bottom)
+		)
+	)
 	(gr_text "CCD"
 		(at 26.67 69.342 0)
@@
 		)
 	)
+	(gr_text "GND"
+		(at 67.679 66.04 180)
+		(layer "F.SilkS")
+		(effects
+			(font
+				(size 0.5 0.5)
+				(thickness 0.125)
+				(bold yes)
+			)
+			(justify left bottom)
+		)
+	)
+	(gr_text "OUT"
+		(at 48.932024 65.913 180)
+		(layer "F.SilkS")
+		(effects
+			(font
+				(size 0.5 0.5)
+				(thickness 0.125)
+				(bold yes)
+			)
+			(justify left bottom)
+		)
+	)
 	(gr_text "Mars Rover Design Team\nMissouri S&T"
 		(at 39.37 87.884 0)
@@
 		)
 	)
+	(gr_text "+5V"
+		(at 47.204 66.04 180)
+		(layer "F.SilkS")
+		(effects
+			(font
+				(size 0.5 0.5)
+				(thickness 0.125)
+				(bold yes)
+			)
+			(justify left bottom)
+		)
+	)
+	(gr_text "CMOS_CLK"
+		(at 53.250024 65.9638 180)
+		(layer "F.SilkS")
+		(effects
+			(font
+				(size 0.5 0.5)
+				(thickness 0.125)
+				(bold yes)
+			)
+			(justify left bottom)
+		)
+	)
+	(gr_text "Trig_OUT"
+		(at 65.786 66.04 180)
+		(layer "F.SilkS")
+		(effects
+			(font
+				(size 0.5 0.5)
+				(thickness 0.125)
+				(bold yes)
+			)
+			(justify left bottom)
+		)
+	)
+	(gr_text "SDI\n"
+		(at 62.343224 66.0654 180)
+		(layer "F.SilkS")
+		(effects
+			(font
+				(size 0.5 0.5)
+				(thickness 0.125)
+				(bold yes)
+			)
+			(justify left bottom)
+		)
+	)
+	(gr_text "ADC_CLK"
+		(at 60.666824 66.05 180)
+		(layer "F.SilkS")
+		(effects
+			(font
+				(size 0.5 0.5)
+				(thickness 0.125)
+				(bold yes)
+			)
+			(justify left bottom)
+		)
+	)
 	(gr_text "CMOS Board, Rev 2\n"
 		(at 39.37 85.598 0)
@@
 				(bold yes)
 			)
+			(justify left bottom)
+		)
+	)
+	(gr_text "ST"
+		(at 56.856824 66.0146 180)
+		(layer "F.SilkS")
+		(effects
+			(font
+				(size 0.5 0.5)
+				(thickness 0.125)
+				(bold yes)
+			)
+			(justify left bottom)
+		)
+	)
+	(gr_text "+3V3"
+		(at 44.704 66.04 180)
+		(layer "F.SilkS")
+		(effects
+			(font
+				(size 0.5 0.5)
+				(thickness 0.125)
+				(bold yes)
+			)

Commit message: Rev2 Fixes
Parts:
- moved C14 15.1 mm to (69.1, 88.4), turned to -90 degrees
- moved U4 5.46 mm to (62.7, 88.9), turned to 180 degrees
- moved C13 4.44 mm to (66.8, 88.4), turned to -90 degrees
- moved R16 3.58 mm to (58.9, 88.6), turned to -90 degrees
- moved R14 2.79 mm to (56.9, 88.6), turned to -90 degrees
- moved R3 1.27 mm to (68.1, 75.7)
- moved R15 0.78 mm to (62.4, 86.4), turned to 180 degrees
- moved C1 0.52 mm to (63.0, 74.9)
- moved R4 0.51 mm to (63.0, 81.0)
Connections:
- C14 pad 1: /ADC/opIND+ -> +5V
- R15 pad 1: Net-(R15-Pad1) -> GND
- R15 pad 2: /ADC/opIND+ -> Net-(R15-Pad2)
- R16 pad 1: GND -> Net-(R15-Pad2)
- R16 pad 2: Net-(R15-Pad1) -> /ADC/opIND+
- U4 pad 4: Net-(R15-Pad1) -> Net-(R15-Pad2)
Routing:
- net +5V: track 128.8 -> 140.0 mm
- net Net-(R15-Pad2): track 0.00 -> 4.61 mm
- net Net-(R15-Pad1): track 4.40 -> 0.00 mm, vias 2 -> 0
- net /ADC/opIND+: track 31.9 -> 28.0 mm, vias 4 -> 2
- net /ADC/SDI: track 39.8 -> 42.1 mm
- net /ADC/CLK2: track 38.1 -> 40.4 mm, vias 4 -> 2
- net Net-(U1-ST): track 1.50 -> 2.77 mm, vias 1 -> 0
- net Net-(U3-AIN+): track 14.5 -> 15.1 mm, vias 4 -> 2
- net /CCD/opINB+: track 29.3 -> 29.9 mm
- net /CCD/CLKb: track 14.0 -> 13.4 mm
- net Net-(Q2-D): track 28.2 -> 27.6 mm
- net /ADC/Video: track 56.9 -> 56.4 mm, vias 6 -> 4
- net Net-(U1-VIcp): track 1.56 -> 2.01 mm, vias 1 -> 0
- net /CCD/STb: track 15.9 -> 15.6 mm, vias 2 -> 0
- net +3V3: track 21.5 -> 21.8 mm, vias 4 -> 2
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Other:
- board text added: "1V8"
- board text added: "5V"
- board text added: "AIN+"
- board text added: "VID"
- board text removed: "2710"
- board text removed: "CCD"
- board text removed: "mils"
- board text removed: "r: 500"
