File: CCD Breakout/ccd.kicad_sch (KiCad schematic)
At the start: 17 parts, among them U1 CCD, U5 74HC541PW_118

Commit message: Rev2 Fixes
Changed lines of the file:
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@@
 	(wire
 		(pts
-			(xy 191.77 35.56) (xy 198.12 35.56)
+			(xy 191.77 35.56) (xy 200.66 35.56)
 		)
 		(stroke
@@
 	(wire
 		(pts
-			(xy 222.25 38.1) (xy 224.79 38.1)
+			(xy 217.17 38.1) (xy 224.79 38.1)
 		)
 		(stroke
@@
 	(wire
 		(pts
-			(xy 264.16 35.56) (xy 270.51 35.56)
+			(xy 265.43 35.56) (xy 270.51 35.56)
 		)
 		(stroke
@@
 	(hierarchical_label "opOUTB"
 		(shape input)
-		(at 222.25 38.1 180)
+		(at 217.17 38.1 180)
 		(effects
 			(font
@@
 	(hierarchical_label "opOUTC"
 		(shape input)
-		(at 264.16 35.56 180)
+		(at 265.43 35.56 180)
 		(effects
 			(font
@@
 	(hierarchical_label "opINB+"
 		(shape output)
-		(at 198.12 35.56 0)
+		(at 200.66 35.56 0)
 		(effects
 			(font
@@
 			)
 		)
-		(property "Datasheet" "74HC541PW_118"
+		(property "Datasheet" "https://assets.nexperia.com/documents/data-sheet/74HC_HCT541.pdf"
 			(at 48.26 39.37 0)
 			(effects

Commit message: Miscellaneous schematic fixes
Connections:
- net opINB+ renamed +1V
Other:
- note added: "CCD"
- note added: "Voltage Shifter (.6v-2.6v -> 0v-5v)"
- moved on the sheet: C7, R6, R9
