File: CCD Breakout/CCD_Breakout.kicad_sch (KiCad schematic)
At the start: 2 parts

Commit message: Finalize board design
Parts:
- added H3, H4: ~, MRDT_Drill_Holes:4_40_Hole_Pad_Via, symbol MRDT_Connectors:4_40_Mounting_Hole_Pad
- H1, H2: footprint MRDT_Drill_Holes:4_40_Hole -> MRDT_Drill_Holes:4_40_Hole_Pad_Via; symbol Mechanical:MountingHole -> MRDT_Connectors:4_40_Mounting_Hole_Pad; now in the parts list
Connections:
- new net GND: H1.1, H2.1, H3.1, H4.1
